Commit message: Cleanup hands to separate out gamma sensor

File: mmint_franka_description/robots/hands/panda_gelslim.xacro (robot description, xacro)
@@ -1,124 +1,106 @@
 <?xml version="1.0" encoding="utf-8"?>
 <robot xmlns:xacro="http://www.ros.org/wiki/xacro" name="panda_gelslim">
-  <xacro:macro name="panda_gelslim" params="connected_to:='' ns:='' rpy:='0 0 0' xyz:='0 0 0'">
-    <xacro:unless value="${connected_to == ''}">
-      <joint name="${ns}_ft_joint" type="fixed">
-        <parent link="${connected_to}"/>
-        <child link="${ns}_ft"/>
-        <origin xyz="${xyz}" rpy="${rpy}"/>
-      </joint>
-    </xacro:unless>
-    <link name="${ns}_ft">
-      <visual>
-        <geometry>
-          <mesh filename="package://mmint_franka_description/meshes/visual/gamma_insert.stl"/>
-        </geometry>
-        <material name="grey"/>
-      </visual>
-      <collision>
-        <geometry>
-          <mesh filename="package://mmint_franka_description/meshes/collision/gamma_insert.stl"/>
-        </geometry>
-      </collision>
-    </link>
-    <joint name="${ns}_hand_joint" type="fixed">
-      <parent link="${ns}_ft"/>
-      <child link="${ns}_hand"/>
-      <origin xyz="0 0 0.0487" rpy="0 0 0"/>
-    </joint>
-    <link name="${ns}_hand">
-      <visual>
-        <geometry>
-          <mesh filename="package://franka_description/meshes/visual/hand.dae"/>
-        </geometry>
-      </visual>
-      <collision>
-        <geometry>
-          <mesh filename="package://franka_description/meshes/collision/hand.stl"/>
-        </geometry>
-      </collision>
-    </link>
-    <link name="${ns}_leftfinger">
-      <visual>
-        <origin rpy="0 0 ${pi}" xyz="0 0.0127025082 0"/>
-        <geometry>
-          <mesh filename="package://mmint_franka_description/meshes/visual/gelslim_3mm.stl"/>
-        </geometry>
-        <material name="grey"/>
-      </visual>
-      <collision>
-        <origin rpy="0 0 ${pi}" xyz="0 0.0127025082 0"/>
-        <geometry>
-          <mesh filename="package://mmint_franka_description/meshes/collision/gelslim_3mm.stl"/>
-        </geometry>
-      </collision>
-    </link>
-    <link name="${ns}_rightfinger">
-      <visual>
-        <origin rpy="0 0 0" xyz="0 -0.0127025082 0"/>
-        <geometry>
-          <mesh filename="package://mmint_franka_description/meshes/visual/gelslim_3mm.stl"/>
-        </geometry>
-        <material name="grey"/>
-      </visual>
-      <collision>
-        <origin rpy="0 0 0" xyz="0 -0.0127025082 0"/>
-        <geometry>
-          <mesh filename="package://mmint_franka_description/meshes/collision/gelslim_3mm.stl"/>
-        </geometry>
-      </collision>
-   </link>
-    <joint name="${ns}_finger_joint1" type="prismatic">
-      <parent link="${ns}_hand"/>
-      <child link="${ns}_leftfinger"/>
-      <origin xyz="0 0 0.0584" rpy="0 0 0"/>
-      <axis xyz="0 1 0"/>
-      <limit effort="20" lower="0.0" upper="0.04" velocity="0.2"/>
-    </joint>
-    <joint name="${ns}_finger_joint2" type="prismatic">
-      <parent link="${ns}_hand"/>
-      <child link="${ns}_rightfinger"/>
-      <origin xyz="0 0 0.0584" rpy="0 0 0"/>
-      <axis xyz="0 -1 0"/>
-      <limit effort="20" lower="0.0" upper="0.04" velocity="0.2"/>
-      <mimic joint="${ns}_finger_joint1" />
-    </joint>
-    <link name="${ns}_left_gelpad_link">
-      <inertial>
-        <origin rpy="0 0 0" xyz="0 0 0"/>
-        <mass value="0.0"/>
-        <inertia ixx="0.1" ixy="0" ixz="0" iyy="0.1" iyz="0" izz="0.1"/>
-      </inertial>
-    </link>
-    <link name="${ns}_right_gelpad_link">
-      <inertial>
-        <origin rpy="0 0 0" xyz="0 0 0"/>
-        <mass value="0.0"/>
-        <inertia ixx="0.1" ixy="0" ixz="0" iyy="0.1" iyz="0" izz="0.1"/>
-      </inertial>
-    </link>
-    <joint name="${ns}_left_gelpad" type="fixed">
-      <parent link="${ns}_leftfinger"/>
-      <child link="${ns}_left_gelpad_link"/>
-      <origin xyz="0 0 0.072" rpy="0 0 0"/>
-    </joint>
-    <joint name="${ns}_right_gelpad" type="fixed">
-      <parent link="${ns}_rightfinger"/>
-      <child link="${ns}_right_gelpad_link"/>
-      <origin xyz="0 0 0.072" rpy="0 0 0"/>
-    </joint>
-    <link name="${ns}_gripper_origin">
-      <inertial>
-        <origin rpy="0 0 0" xyz="0 0 0"/>
-        <mass value="0.0"/>
-        <inertia ixx="0.1" ixy="0" ixz="0" iyy="0.1" iyz="0" izz="0.1"/>
-      </inertial>
-    </link>
-    <joint name="${ns}_gripper" type="fixed">
-      <parent link="${ns}_hand"/>
-      <child link="${ns}_gripper_origin"/>
-<!--      <origin rpy="0 0 0" xyz="0 0 0.1264"/>-->
-      <origin rpy="0 0 0" xyz="0 0 0.1304"/>
-    </joint>
-  </xacro:macro>
+    <xacro:include filename="$(find mmint_franka_description)/robots/hands/gamma.xacro"/>
+    <xacro:macro name="panda_gelslim" params="connected_to:='' ns:='' rpy:='0 0 0' xyz:='0 0 0'">
+        <xacro:gamma ns="${ns}" connected_to="${connected_to}" rpy="${rpy}" xyz="${xyz}"/>
+        <joint name="${ns}_hand_joint" type="fixed">
+            <parent link="${ns}_ft_origin"/>
+            <child link="${ns}_hand"/>
+            <origin xyz="0 0 0.0079" rpy="0 0 0"/>
+        </joint>
+        <link name="${ns}_hand">
+            <visual>
+                <geometry>
+                    <mesh filename="package://franka_description/meshes/visual/hand.dae"/>
+                </geometry>
+            </visual>
+            <collision>
+                <geometry>
+                    <mesh filename="package://franka_description/meshes/collision/hand.stl"/>
+                </geometry>
+            </collision>
+        </link>
+        <link name="${ns}_leftfinger">
+            <visual>
+                <origin rpy="0 0 ${pi}" xyz="0 0.0127025082 0"/>
+                <geometry>
+                    <mesh filename="package://mmint_franka_description/meshes/visual/gelslim_3mm.stl"/>
+                </geometry>
+                <material name="grey"/>
+            </visual>
+            <collision>
+                <origin rpy="0 0 ${pi}" xyz="0 0.0127025082 0"/>
+                <geometry>
+                    <mesh filename="package://mmint_franka_description/meshes/collision/gelslim_3mm.stl"/>
+                </geometry>
+            </collision>
+        </link>
+        <link name="${ns}_rightfinger">
+            <visual>
+                <origin rpy="0 0 0" xyz="0 -0.0127025082 0"/>
+                <geometry>
+                    <mesh filename="package://mmint_franka_description/meshes/visual/gelslim_3mm.stl"/>
+                </geometry>
+                <material name="grey"/>
+            </visual>
+            <collision>
+                <origin rpy="0 0 0" xyz="0 -0.0127025082 0"/>
+                <geometry>
+                    <mesh filename="package://mmint_franka_description/meshes/collision/gelslim_3mm.stl"/>
+                </geometry>
+            </collision>
+        </link>
+        <joint name="${ns}_finger_joint1" type="prismatic">
+            <parent link="${ns}_hand"/>
+            <child link="${ns}_leftfinger"/>
+            <origin xyz="0 0 0.0584" rpy="0 0 0"/>
+            <axis xyz="0 1 0"/>
+            <limit effort="20" lower="0.0" upper="0.04" velocity="0.2"/>
+        </joint>
+        <joint name="${ns}_finger_joint2" type="prismatic">
+            <parent link="${ns}_hand"/>
+            <child link="${ns}_rightfinger"/>
+            <origin xyz="0 0 0.0584" rpy="0 0 0"/>
+            <axis xyz="0 -1 0"/>
+            <limit effort="20" lower="0.0" upper="0.04" velocity="0.2"/>
+            <mimic joint="${ns}_finger_joint1"/>
+        </joint>
+        <link name="${ns}_left_gelpad_link">
+            <inertial>
+                <origin rpy="0 0 0" xyz="0 0 0"/>
+                <mass value="0.0"/>
+                <inertia ixx="0.1" ixy="0" ixz="0" iyy="0.1" iyz="0" izz="0.1"/>
+            </inertial>
+        </link>
+        <link name="${ns}_right_gelpad_link">
+            <inertial>
+                <origin rpy="0 0 0" xyz="0 0 0"/>
+                <mass value="0.0"/>
+                <inertia ixx="0.1" ixy="0" ixz="0" iyy="0.1" iyz="0" izz="0.1"/>
+            </inertial>
+        </link>
+        <joint name="${ns}_left_gelpad" type="fixed">
+            <parent link="${ns}_leftfinger"/>
+            <child link="${ns}_left_gelpad_link"/>
+            <origin xyz="0 0 0.072" rpy="0 0 0"/>
+        </joint>
+        <joint name="${ns}_right_gelpad" type="fixed">
+            <parent link="${ns}_rightfinger"/>
+            <child link="${ns}_right_gelpad_link"/>
+            <origin xyz="0 0 0.072" rpy="0 0 0"/>
+        </joint>
+        <link name="${ns}_gripper_origin">
+            <inertial>
+                <origin rpy="0 0 0" xyz="0 0 0"/>
+                <mass value="0.0"/>
+                <inertia ixx="0.1" ixy="0" ixz="0" iyy="0.1" iyz="0" izz="0.1"/>
+            </inertial>
+        </link>
+        <joint name="${ns}_gripper" type="fixed">
+            <parent link="${ns}_hand"/>
+            <child link="${ns}_gripper_origin"/>
+            <!--      <origin rpy="0 0 0" xyz="0 0 0.1264"/>-->
+            <origin rpy="0 0 0" xyz="0 0 0.1304"/>
+        </joint>
+    </xacro:macro>
 </robot>

File: mmint_franka_description/robots/hands/panda_hand.xacro (robot description, xacro)
@@ -1,105 +1,81 @@
 <?xml version="1.0" encoding="utf-8"?>
 <robot xmlns:xacro="http://www.ros.org/wiki/xacro" name="panda_hand">
-  <xacro:macro name="panda_hand" params="connected_to:='' ns:='' rpy:='0 0 0' xyz:='0 0 0'">
-    <xacro:unless value="${connected_to == ''}">
-      <joint name="${ns}_ft_joint" type="fixed">
-        <parent link="${connected_to}"/>
-        <child link="${ns}_ft"/>
-        <origin xyz="${xyz}" rpy="${rpy}"/>
-      </joint>
-    </xacro:unless>
-    <link name="${ns}_ft">
-      <visual>
-        <geometry>
-          <mesh filename="package://mmint_franka_description/meshes/visual/gamma_insert.stl"/>
-        </geometry>
-        <material name="grey"/>
-      </visual>
-      <collision>
-        <geometry>
-          <mesh filename="package://mmint_franka_description/meshes/collision/gamma_insert.stl"/>
-        </geometry>
-      </collision>
-    </link>
-    <link name="${ns}_ft_origin"/>
-    <joint name="${ns}_ft_origin_joint" type="fixed">
-      <parent link="${ns}_ft"/>
-      <child link="${ns}_ft_origin"/>
-      <origin xyz="0 0 0.0408" rpy="0 0 0"/>
-    </joint>
-    <joint name="${ns}_hand_joint" type="fixed">
-      <parent link="${ns}_ft_origin"/>
-      <child link="${ns}_hand"/>
-      <origin xyz="0 0 0.0079" rpy="0 0 0"/>
-    </joint>
-    <link name="${ns}_hand">
-      <visual>
-        <geometry>
-          <mesh filename="package://franka_description/meshes/visual/hand.dae"/>
-        </geometry>
-      </visual>
-      <collision>
-        <geometry>
-          <mesh filename="package://franka_description/meshes/collision/hand.stl"/>
-        </geometry>
-      </collision>
-    </link>
-    <link name="${ns}_leftfinger">
-      <visual>
-        <origin rpy="0 0 0" xyz="0 0.01325 0"/>
-        <geometry>
-          <mesh filename="package://mmint_franka_description/meshes/visual/knuckle.stl"/>
-        </geometry>
-        <material name="grey"/>
-      </visual>
-      <collision>
-        <origin rpy="0 0 0" xyz="0 0.01325 0"/>
-        <geometry>
-          <mesh filename="package://mmint_franka_description/meshes/collision/knuckle.stl"/>
-        </geometry>
-      </collision>
-    </link>
-    <link name="${ns}_rightfinger">
-      <visual>
-        <origin rpy="0 0 ${pi}" xyz="0 -0.01325 0"/>
-        <geometry>
-          <mesh filename="package://mmint_franka_description/meshes/visual/knuckle.stl"/>
-        </geometry>
-        <material name="grey"/>
-      </visual>
-      <collision>
-        <origin rpy="0 0 ${pi}" xyz="0 -0.01325 0"/>
-        <geometry>
-          <mesh filename="package://mmint_franka_description/meshes/collision/knuckle.stl"/>
-        </geometry>
-      </collision>
-   </link>
-    <joint name="${ns}_finger_joint1" type="prismatic">
-      <parent link="${ns}_hand"/>
-      <child link="${ns}_leftfinger"/>
-      <origin xyz="0 0 0.0584" rpy="0 0 0"/>
-      <axis xyz="0 1 0"/>
-      <limit effort="20" lower="0.0" upper="0.04" velocity="0.2"/>
-    </joint>
-    <joint name="${ns}_finger_joint2" type="prismatic">
-      <parent link="${ns}_hand"/>
-      <child link="${ns}_rightfinger"/>
-      <origin xyz="0 0 0.0584" rpy="0 0 0"/>
-      <axis xyz="0 -1 0"/>
-      <limit effort="20" lower="0.0" upper="0.04" velocity="0.2"/>
-      <mimic joint="${ns}_finger_joint1" />
-    </joint>
-    <link name="${ns}_gripper_origin">
-      <inertial>
-        <origin rpy="0 0 0" xyz="0 0 0"/>
-        <mass value="0.0"/>
-        <inertia ixx="0.1" ixy="0" ixz="0" iyy="0.1" iyz="0" izz="0.1"/>
-      </inertial>
-    </link>
-    <joint name="${ns}_gripper" type="fixed">
-      <parent link="${ns}_hand"/>
-      <child link="${ns}_gripper_origin"/>
-      <origin rpy="0 0 0" xyz="0 0 0.1034"/>
-    </joint>
-  </xacro:macro>
+    <xacro:include filename="$(find mmint_franka_description)/robots/hands/gamma.xacro"/>
+    <xacro:macro name="panda_hand" params="connected_to:='' ns:='' rpy:='0 0 0' xyz:='0 0 0'">
+        <xacro:gamma ns="${ns}" connected_to="${connected_to}" rpy="${rpy}" xyz="${xyz}"/>
+        <joint name="${ns}_hand_joint" type="fixed">
+            <parent link="${ns}_ft_origin"/>
+            <child link="${ns}_hand"/>
+            <origin xyz="0 0 0.0079" rpy="0 0 0"/>
+        </joint>
+        <link name="${ns}_hand">
+            <visual>
+                <geometry>
+                    <mesh filename="package://franka_description/meshes/visual/hand.dae"/>
+                </geometry>
+            </visual>
+            <collision>
+                <geometry>
+                    <mesh filename="package://franka_description/meshes/collision/hand.stl"/>
+                </geometry>
+            </collision>
+        </link>
+        <link name="${ns}_leftfinger">
+            <visual>
+                <origin rpy="0 0 0" xyz="0 0.01325 0"/>
+                <geometry>
+                    <mesh filename="package://mmint_franka_description/meshes/visual/knuckle.stl"/>
+                </geometry>
+                <material name="grey"/>
+            </visual>
+            <collision>
+                <origin rpy="0 0 0" xyz="0 0.01325 0"/>
+                <geometry>
+                    <mesh filename="package://mmint_franka_description/meshes/collision/knuckle.stl"/>
+                </geometry>
+            </collision>
+        </link>
+        <link name="${ns}_rightfinger">
+            <visual>
+                <origin rpy="0 0 ${pi}" xyz="0 -0.01325 0"/>
+                <geometry>
+                    <mesh filename="package://mmint_franka_description/meshes/visual/knuckle.stl"/>
+                </geometry>
+                <material name="grey"/>
+            </visual>
+            <collision>
+                <origin rpy="0 0 ${pi}" xyz="0 -0.01325 0"/>
+                <geometry>
+                    <mesh filename="package://mmint_franka_description/meshes/collision/knuckle.stl"/>
+                </geometry>
+            </collision>
+        </link>
+        <joint name="${ns}_finger_joint1" type="prismatic">
+            <parent link="${ns}_hand"/>
+            <child link="${ns}_leftfinger"/>
+            <origin xyz="0 0 0.0584" rpy="0 0 0"/>
+            <axis xyz="0 1 0"/>
+            <limit effort="20" lower="0.0" upper="0.04" velocity="0.2"/>
+        </joint>
+        <joint name="${ns}_finger_joint2" type="prismatic">
+            <parent link="${ns}_hand"/>
+            <child link="${ns}_rightfinger"/>
+            <origin xyz="0 0 0.0584" rpy="0 0 0"/>
+            <axis xyz="0 -1 0"/>
+            <limit effort="20" lower="0.0" upper="0.04" velocity="0.2"/>
+            <mimic joint="${ns}_finger_joint1"/>
+        </joint>
+        <link name="${ns}_gripper_origin">
+            <inertial>
+                <origin rpy="0 0 0" xyz="0 0 0"/>
+                <mass value="0.0"/>
+                <inertia ixx="0.1" ixy="0" ixz="0" iyy="0.1" iyz="0" izz="0.1"/>
+            </inertial>
+        </link>
+        <joint name="${ns}_gripper" type="fixed">
+            <parent link="${ns}_hand"/>
+            <child link="${ns}_gripper_origin"/>
+            <origin rpy="0 0 0" xyz="0 0 0.1034"/>
+        </joint>
+    </xacro:macro>
 </robot>

File: mmint_franka_description/robots/mmint_combined_panda.urdf.xacro (robot description, xacro)
@@ -48,6 +48,6 @@
         <xacro:panda_gelslim ns="$(arg arm_id_1)" rpy="0 0 ${-pi/4}" connected_to="$(arg arm_id_1)_link8"/>
     </xacro:if>
-    <xacro:if value="${hand_1 == 'panda_ft'}">
-        <xacro:panda_ft ns="$(arg arm_id_1)" rpy="0 0 ${-pi/4}" connected_to="$(arg arm_id_1)_link8"/>
+    <xacro:if value="${hand_1 == 'gamma'}">
+        <xacro:gamma ns="$(arg arm_id_1)" rpy="0 0 ${-pi/4}" connected_to="$(arg arm_id_1)_link8"/>
     </xacro:if>
     <!-- Load right arm -->
@@ -60,6 +60,6 @@
         <xacro:panda_gelslim ns="$(arg arm_id_2)" rpy="0 0 ${-pi/4}" connected_to="$(arg arm_id_2)_link8"/>
     </xacro:if>
-    <xacro:if value="${hand_2 == 'panda_ft'}">
-        <xacro:panda_ft ns="$(arg arm_id_2)" rpy="0 0 ${-pi/4}" connected_to="$(arg arm_id_2)_link8"/>
+    <xacro:if value="${hand_2 == 'gamma'}">
+        <xacro:gamma ns="$(arg arm_id_1)" rpy="0 0 ${-pi/4}" connected_to="$(arg arm_id_1)_link8"/>
     </xacro:if>
 </robot>
