Commit message: Add new flange adapter for sponge setup

File: mmint_franka_description/robots/hands/sponge_eef.xacro (robot description, xacro)
@@ -1,5 +1,6 @@
 <?xml version="1.0" encoding="utf-8"?>
 <robot xmlns:xacro="http://www.ros.org/wiki/xacro" name="sponge_eef">
-    <xacro:macro name="sponge_eef" params="connected_to:='' ns:='' rpy:='0 0 0' xyz:='0 0 0' extend:=${True}">
+    <xacro:macro name="sponge_eef"
+                 params="connected_to:='' ns:='' rpy:='0 0 0' xyz:='0 0 0' gamma_:=${True} extend:=${True}">
         <xacro:unless value="${connected_to == ''}">
             <joint name="${ns}_ft_joint" type="fixed">
@@ -9,23 +10,46 @@
             </joint>
         </xacro:unless>
-        <link name="${ns}_ft">
-            <visual>
-                <geometry>
-                    <mesh filename="package://mmint_franka_description/meshes/visual/gamma_insert_v2.stl"/>
-                </geometry>
-                <material name="grey"/>
-            </visual>
-            <collision>
-                <geometry>
-                    <mesh filename="package://mmint_franka_description/meshes/collision/gamma_insert_v2.stl"/>
-                </geometry>
-            </collision>
-        </link>
-        <link name="${ns}_ft_origin"/>
-        <joint name="${ns}_ft_origin_joint" type="fixed">
-            <parent link="${ns}_ft"/>
-            <child link="${ns}_ft_origin"/>
-            <origin xyz="0 0 0.0408" rpy="0 0 0"/>
-        </joint>
+        <xacro:if value="${gamma_}">
+            <link name="${ns}_ft">
+                <visual>
+                    <geometry>
+                        <mesh filename="package://mmint_franka_description/meshes/visual/gamma_insert_v2.stl"/>
+                    </geometry>
+                    <material name="grey"/>
+                </visual>
+                <collision>
+                    <geometry>
+                        <mesh filename="package://mmint_franka_description/meshes/collision/gamma_insert_v2.stl"/>
+                    </geometry>
+                </collision>
+            </link>
+            <link name="${ns}_ft_origin"/>
+            <joint name="${ns}_ft_origin_joint" type="fixed">
+                <parent link="${ns}_ft"/>
+                <child link="${ns}_ft_origin"/>
+                <origin xyz="0 0 0.0408" rpy="0 0 0"/>
+            </joint>
+        </xacro:if>
+        <xacro:unless value="${gamma_}">
+            <link name="${ns}_ft">
+                <visual>
+                    <geometry>
+                        <mesh filename="package://mmint_franka_description/meshes/visual/flange_adapter.stl" scale="0.001 0.001 0.001"/>
+                    </geometry>
+                    <material name="grey"/>
+                </visual>
+                <collision>
+                    <geometry>
+                        <mesh filename="package://mmint_franka_description/meshes/visual/flange_adapter.stl" scale="0.001 0.001 0.001"/>
+                    </geometry>
+                </collision>
+            </link>
+            <link name="${ns}_ft_origin"/>
+            <joint name="${ns}_ft_origin_joint" type="fixed">
+                <parent link="${ns}_ft"/>
+                <child link="${ns}_ft_origin"/>
+                <origin xyz="0 0 0.036" rpy="0 0 0"/>
+            </joint>
+        </xacro:unless>
         <link name="${ns}_mount">
             <visual>

File: mmint_franka_description/robots/mmint_combined_panda.urdf.xacro (robot description, xacro)
@@ -60,4 +60,8 @@
                           extend="${True}"/>
     </xacro:if>
+    <xacro:if value="${hand_1 == 'sponge_eef_extend_no_gamma'}">
+        <xacro:sponge_eef ns="$(arg arm_id_1)" rpy="0 0 ${-pi/4}" connected_to="$(arg arm_id_1)_link8" extend="${True}"
+                          gamma_="${False}"/>
+    </xacro:if>
     <!-- Load right arm -->
     <xacro:franka_arm arm_id="$(arg arm_id_2)" connected_to="base" xyz="-0.2815 0.0 0.6" rpy="0 0 0"
@@ -83,3 +87,7 @@
                           extend="${True}"/>
     </xacro:if>
+    <xacro:if value="${hand_2 == 'sponge_eef_extend_no_gamma'}">
+        <xacro:sponge_eef ns="$(arg arm_id_2)" rpy="0 0 ${-pi/4}" connected_to="$(arg arm_id_2)_link8" extend="${True}"
+                          gamma_="${False}"/>
+    </xacro:if>
 </robot>

File: mmint_franka_description/robots/panda.urdf (robot description, URDF)
Before this commit: robot panda, 48 links, 47 joints
Links:
- removed link panda_1_gripper_origin
- removed link panda_1_hand
- removed link panda_1_leftfinger
- removed link panda_1_rightfinger
- removed link panda_2_ft
- removed link panda_2_ft_origin
- removed link panda_2_gripper_origin
- removed link panda_2_hand
- removed link panda_2_leftfinger
- removed link panda_2_rightfinger
- added link panda_1_mount; collision cylinder length=0.036 radius=0.03; visual mesh filename=package://mmint_franka_description/meshes/visual/sponge_mou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
- added link panda_1_mount_extend; collision mesh filename=package://mmint_franka_description/meshes/collision/mount_e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; visual mesh filename=package://mmint_franka_description/meshes/visual/mount_exte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
- added link panda_1_sponge
- link panda_1_ft: geometry collision mesh filename=package://mmint_franka_description/meshes/visual/flange_ada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 scale=0.001 0.001 0.001; visual mesh filename=package://mmint_franka_description/meshes/visual/flange_ada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 scale=0.001 0.001 0.001
Joints:
- removed joint panda_1_finger_joint1
- removed joint panda_1_finger_joint2
- removed joint panda_1_gripper
- removed joint panda_1_hand_joint
- removed joint panda_2_finger_joint1
- removed joint panda_2_finger_joint2
- removed joint panda_2_ft_joint
- removed joint panda_2_ft_origin_joint
- removed joint panda_2_gripper
- removed joint panda_2_hand_joint
- added joint panda_1_mount_extend_joint: type fixed, parent panda_1_ft_origin, child panda_1_mount_extend, origin xyz=0 0 0 rpy=0 0 0
- added joint panda_1_mount_joint: type fixed, parent panda_1_mount_extend, child panda_1_mount, origin xyz=0.01333 0 0.05219 rpy=0.0 0.7853981609493879 0.0
- added joint panda_1_mount_sponge_joint: type fixed, parent panda_1_mount, child panda_1_sponge, origin xyz=0 0 0.036 rpy=0 0 0
- joint panda_1_ft_origin_joint: origin xyz=0 0 0.0408 rpy=0 0 0 -> xyz=0 0 0.036 rpy=0 0 0

File: mmint_franka_moveit_config/config/panda.srdf.xacro (robot description, xacro)
@@ -27,5 +27,5 @@
         </group>
     </xacro:if>
-    <xacro:if value="${hand_1 == 'sponge_eef' or hand_1 == 'sponge_eef_extend'}">
+    <xacro:if value="${hand_1 == 'sponge_eef' or hand_1 == 'sponge_eef_extend' or hand_1 == 'sponge_eef_extend_no_gamma'}">
         <group name="$(arg arm_id_1)">
             <chain base_link="$(arg arm_id_1)_link0" tip_link="$(arg arm_id_1)_mount"/>
@@ -33,5 +33,5 @@
     </xacro:if>
     <xacro:unless
-            value="${hand_1 == 'panda_hand' or hand_1 == 'panda_hand_no_gamma' or hand_1 == 'panda_gelslim' or hand_1 == 'gamma' or hand_1 == 'sponge_eef' or hand_1 == 'sponge_eef_extend'}">
+            value="${hand_1 == 'panda_hand' or hand_1 == 'panda_hand_no_gamma' or hand_1 == 'panda_gelslim' or hand_1 == 'gamma' or hand_1 == 'sponge_eef' or hand_1 == 'sponge_eef_extend' or hand_1 == 'sponge_eef_extend_no_gamma'}">
         <group name="$(arg arm_id_1)">
             <chain base_link="$(arg arm_id_1)_link0" tip_link="$(arg arm_id_1)_link8"/>
@@ -48,5 +48,5 @@
         </group>
     </xacro:if>
-    <xacro:if value="${hand_2 == 'sponge_eef' or hand_2 == 'sponge_eef_extend'}">
+    <xacro:if value="${hand_2 == 'sponge_eef' or hand_2 == 'sponge_eef_extend' or hand_2 == 'sponge_eef_extend_no_gamma'}">
         <group name="$(arg arm_id_2)">
             <chain base_link="$(arg arm_id_2)_link0" tip_link="$(arg arm_id_2)_mount"/>
@@ -54,5 +54,5 @@
     </xacro:if>
     <xacro:unless
-            value="${hand_2 == 'panda_hand' or hand_2 == 'panda_hand_no_gamma' or hand_2 == 'panda_gelslim' or hand_2 == 'gamma' or hand_2 == 'sponge_eef' or hand_2 == 'sponge_eef_extend'}">
+            value="${hand_2 == 'panda_hand' or hand_2 == 'panda_hand_no_gamma' or hand_2 == 'panda_gelslim' or hand_2 == 'gamma' or hand_2 == 'sponge_eef' or hand_2 == 'sponge_eef_extend' or hand_2 == 'sponge_eef_extend_no_gamma'}">
         <group name="$(arg arm_id_2)">
             <chain base_link="$(arg arm_id_2)_link0" tip_link="$(arg arm_id_2)_link8"/>
@@ -170,5 +170,5 @@
         <disable_collisions link1="$(arg arm_id_1)_ft" link2="$(arg arm_id_1)_mount" reason="Adjacent"/>
     </xacro:if>
-    <xacro:if value="${hand_1 == 'sponge_eef_extend'}">
+    <xacro:if value="${hand_1 == 'sponge_eef_extend' or hand_1 == 'sponge_eef_extend_no_gamma'}">
         <disable_collisions link1="$(arg arm_id_1)_ft" link2="$(arg arm_id_1)_link7_sc" reason="Adjacent"/>
         <disable_collisions link1="$(arg arm_id_1)_ft" link2="$(arg arm_id_1)_mount_extend" reason="Adjacent"/>
@@ -195,5 +195,5 @@
         <disable_collisions link1="$(arg arm_id_2)_ft" link2="$(arg arm_id_2)_mount" reason="Adjacent"/>
     </xacro:if>
-    <xacro:if value="${hand_2 == 'sponge_eef_extend'}">
+    <xacro:if value="${hand_2 == 'sponge_eef_extend' or hand_2 == 'sponge_eef_extend_no_gamma'}">
         <disable_collisions link1="$(arg arm_id_2)_ft" link2="$(arg arm_id_2)_link7_sc" reason="Adjacent"/>
         <disable_collisions link1="$(arg arm_id_2)_ft" link2="$(arg arm_id_2)_mount_extend" reason="Adjacent"/>
