Commit message: jelslim

File: mmint_franka_description/robots/hands/gamma.xacro (robot description, xacro)
@@ -1,3 +1,3 @@
-<?xml version="1.0" encoding="utf-8"?>
+<!-- <?xml version="1.0" encoding="utf-8"?>
 <robot xmlns:xacro="http://www.ros.org/wiki/xacro" name="panda_hand">
     <xacro:macro name="gamma" params="connected_to:='' ns:='' rpy:='0 0 0' xyz:='0 0 0'">
@@ -29,3 +29,3 @@
         </joint>
     </xacro:macro>
-</robot>
+</robot> -->

File: mmint_franka_description/robots/hands/panda_gelslim.xacro (robot description, xacro)
@@ -1,11 +1,11 @@
 <?xml version="1.0" encoding="utf-8"?>
 <robot xmlns:xacro="http://www.ros.org/wiki/xacro" name="panda_gelslim">
-    <xacro:include filename="$(find mmint_franka_description)/robots/hands/gamma.xacro"/>
+    <!-- <xacro:include filename="$(find mmint_franka_description)/robots/hands/gamma.xacro"/> -->
     <xacro:macro name="panda_gelslim" params="connected_to:='' ns:='' rpy:='0 0 0' xyz:='0 0 0'">
-        <xacro:gamma ns="${ns}" connected_to="${connected_to}" rpy="${rpy}" xyz="${xyz}"/>
+        <!-- <xacro:gamma ns="${ns}" connected_to="${connected_to}" rpy="${rpy}" xyz="${xyz}"/> -->
         <joint name="${ns}_hand_joint" type="fixed">
-            <parent link="${ns}_ft_origin"/>
+            <parent link="${ns}_link8"/>
             <child link="${ns}_hand"/>
-            <origin xyz="0 0 0.0079" rpy="0 0 0"/>
+            <origin xyz="0 0 0.0079" rpy="0 0 ${-pi/4}"/>
         </joint>
         <link name="${ns}_hand">
@@ -23,14 +23,14 @@
         <link name="${ns}_leftfinger">
             <visual>
-                <origin rpy="0 0 ${pi}" xyz="0 0.0127025082 0"/>
+                <origin rpy="0 ${pi/2} 0" xyz="-0.016 0 0.055"/>
                 <geometry>
-                    <mesh filename="package://mmint_franka_description/meshes/visual/gelslim_3mm.stl"/>
+                    <mesh scale="2.18216727e-9 2.18216727e-9 2.18216727e-9" filename="package://mmint_franka_description/meshes/visual/gelslim_backup.stl"/>
                 </geometry>
                 <material name="grey"/>
             </visual>
             <collision>
-                <origin rpy="0 0 ${pi}" xyz="0 0.0127025082 0"/>
+                <origin rpy="0 ${pi/2} 0" xyz="-0.016 0 0.055"/>
                 <geometry>
-                    <mesh filename="package://mmint_franka_description/meshes/collision/gelslim_3mm.stl"/>
+                    <mesh scale="2.18216727e-9 2.18216727e-9 2.18216727e-9" filename="package://mmint_franka_description/meshes/collision/gelslim_backup.stl"/>
                 </geometry>
             </collision>
@@ -38,14 +38,14 @@
         <link name="${ns}_rightfinger">
             <visual>
-                <origin rpy="0 0 0" xyz="0 -0.0127025082 0"/>
+                <origin rpy="0 ${pi/2} ${pi}" xyz="0.016 0 0.055"/>
                 <geometry>
-                    <mesh filename="package://mmint_franka_description/meshes/visual/gelslim_3mm.stl"/>
+                    <mesh scale="2.18216727e-9 2.18216727e-9 2.18216727e-9" filename="package://mmint_franka_description/meshes/visual/gelslim_backup.stl"/>
                 </geometry>
                 <material name="grey"/>
             </visual>
             <collision>
-                <origin rpy="0 0 0" xyz="0 -0.0127025082 0"/>
+                <origin rpy="0 ${pi/2} ${pi}" xyz="0.016 0 0.055"/>
                 <geometry>
-                    <mesh filename="package://mmint_franka_description/meshes/collision/gelslim_3mm.stl"/>
+                    <mesh scale="2.18216727e-9 2.18216727e-9 2.18216727e-9" filename="package://mmint_franka_description/meshes/collision/gelslim_backup.stl"/>
                 </geometry>
             </collision>
@@ -83,14 +83,14 @@
             <parent link="${ns}_leftfinger"/>
             <child link="${ns}_left_gelpad_link"/>
-            <origin xyz="0 0 0.072" rpy="0 0 0"/>
+            <origin xyz="0 0 0.06" rpy="0 0 0"/>
         </joint>
         <joint name="${ns}_right_gelpad" type="fixed">
             <parent link="${ns}_rightfinger"/>
             <child link="${ns}_right_gelpad_link"/>
-            <origin xyz="0 0 0.072" rpy="0 0 0"/>
+            <origin xyz="0 0 0.06" rpy="0 0 0"/>
         </joint>
         <link name="${ns}_gripper_origin">
             <inertial>
-                <origin rpy="0 0 0" xyz="0 0 0"/>
+                <origin rpy="0 0 0" xyz="0 0 -0.012"/>
                 <mass value="0.0"/>
                 <inertia ixx="0.1" ixy="0" ixz="0" iyy="0.1" iyz="0" izz="0.1"/>

File: mmint_franka_description/robots/hands/panda_hand.xacro (robot description, xacro)
@@ -1,9 +1,9 @@
 <?xml version="1.0" encoding="utf-8"?>
 <robot xmlns:xacro="http://www.ros.org/wiki/xacro" name="panda_hand">
-    <xacro:include filename="$(find mmint_franka_description)/robots/hands/gamma.xacro"/>
+    <!-- <xacro:include filename="$(find mmint_franka_description)/robots/hands/gamma.xacro"/> -->
     <xacro:macro name="panda_hand" params="connected_to:='' ns:='' rpy:='0 0 0' xyz:='0 0 0'">
-        <xacro:gamma ns="${ns}" connected_to="${connected_to}" rpy="${rpy}" xyz="${xyz}"/>
+        <!-- <xacro:gamma ns="${ns}" connected_to="${connected_to}" rpy="${rpy}" xyz="${xyz}"/> -->
         <joint name="${ns}_hand_joint" type="fixed">
-            <parent link="${ns}_ft_origin"/>
+            <parent link="${ns}_link8"/>
             <child link="${ns}_hand"/>
             <origin xyz="0 0 0.0079" rpy="0 0 0"/>

File: mmint_franka_description/robots/mmint_combined_panda.urdf.xacro (robot description, xacro)
@@ -10,6 +10,6 @@
     <xacro:include filename="$(find mmint_franka_description)/robots/materials.xacro"/>
     <xacro:include filename="$(find franka_description)/robots/common/franka_arm.xacro"/>
-    <xacro:include filename="$(find mmint_franka_description)/robots/hands/gamma.xacro"/>
-    <xacro:include filename="$(find mmint_franka_description)/robots/hands/panda_hand.xacro"/>
+    <!-- <xacro:include filename="$(find mmint_franka_description)/robots/hands/gamma.xacro"/> -->
+    <!-- <xacro:include filename="$(find mmint_franka_description)/robots/hands/panda_hand.xacro"/> -->
     <xacro:include filename="$(find mmint_franka_description)/robots/hands/panda_gelslim.xacro"/>
     <!-- box shaped table as base for the 2 Pandas -->
@@ -45,7 +45,7 @@
         <xacro:panda_gelslim ns="$(arg arm_id_1)" rpy="0 0 ${-pi/4}" connected_to="$(arg arm_id_1)_link8"/>
     </xacro:if>
-    <xacro:if value="${hand_1 == 'gamma'}">
+    <!-- <xacro:if value="${hand_1 == 'gamma'}">
         <xacro:gamma ns="$(arg arm_id_1)" rpy="0 0 ${-pi/4}" connected_to="$(arg arm_id_1)_link8"/>
-    </xacro:if>
+    </xacro:if> -->
     <!-- Load right arm -->
     <xacro:franka_arm arm_id="$(arg arm_id_2)" connected_to="base" xyz="-0.2815 0.0 0.6" rpy="0 0 0"
@@ -57,6 +57,6 @@
         <xacro:panda_gelslim ns="$(arg arm_id_2)" rpy="0 0 ${-pi/4}" connected_to="$(arg arm_id_2)_link8"/>
     </xacro:if>
-    <xacro:if value="${hand_2 == 'gamma'}">
+    <!-- <xacro:if value="${hand_2 == 'gamma'}">
         <xacro:gamma ns="$(arg arm_id_2)" rpy="0 0 ${-pi/4}" connected_to="$(arg arm_id_2)_link8"/>
-    </xacro:if>
+    </xacro:if> -->
 </robot>
