Commit message: Add option to turn off gamma

File: mmint_franka_description/robots/hands/panda_hand.xacro (robot description, xacro)
@@ -2,11 +2,21 @@
 <robot xmlns:xacro="http://www.ros.org/wiki/xacro" name="panda_hand">
     <xacro:include filename="$(find mmint_franka_description)/robots/hands/gamma.xacro"/>
-    <xacro:macro name="panda_hand" params="connected_to:='' ns:='' rpy:='0 0 0' xyz:='0 0 0'">
-        <xacro:gamma ns="${ns}" connected_to="${connected_to}" rpy="${rpy}" xyz="${xyz}"/>
-        <joint name="${ns}_hand_joint" type="fixed">
-            <parent link="${ns}_ft_origin"/>
-            <child link="${ns}_hand"/>
-            <origin xyz="0 0 0.0079" rpy="0 0 0"/>
-        </joint>
+    <xacro:macro name="panda_hand" params="connected_to:='' ns:='' rpy:='0 0 0' xyz:='0 0 0' link:='gamma'">
+        <xacro:if value="${link == 'gamma'}">
+            <xacro:gamma ns="${ns}" connected_to="${connected_to}" rpy="${rpy}" xyz="${xyz}"/>
+            <joint name="${ns}_hand_joint" type="fixed">
+                <parent link="${ns}_ft_origin"/>
+                <child link="${ns}_hand"/>
+                <origin xyz="0 0 0.0079" rpy="0 0 0"/>
+            </joint>
+        </xacro:if>
+        <xacro:unless value="${link == 'gamma'}">
+            <joint name="${ns}_hand_joint" type="fixed">
+                <parent link="${connected_to}"/>
+                <child link="${ns}_hand"/>
+                <origin xyz="${xyz}" rpy="${rpy}"/>
+            </joint>
+        </xacro:unless>
+        <!--        <xacro:gamma ns="${ns}" connected_to="${connected_to}" rpy="${rpy}" xyz="${xyz}"/>-->
         <link name="${ns}_hand">
             <visual>

File: mmint_franka_description/robots/mmint_combined_panda.urdf.xacro (robot description, xacro)
@@ -43,4 +43,7 @@
         <xacro:panda_hand ns="$(arg arm_id_1)" rpy="0 0 ${-pi/4}" connected_to="$(arg arm_id_1)_link8"/>
     </xacro:if>
+    <xacro:if value="${hand_1 == 'panda_hand_no_gamma'}">
+        <xacro:panda_hand ns="$(arg arm_id_1)" rpy="0 0 ${-pi/4}" connected_to="$(arg arm_id_1)_link8" link="no_gamma"/>
+    </xacro:if>
     <xacro:if value="${hand_1 == 'panda_gelslim'}">
         <xacro:panda_gelslim ns="$(arg arm_id_1)" rpy="0 0 ${-pi/4}" connected_to="$(arg arm_id_1)_link8"/>
@@ -63,4 +66,7 @@
         <xacro:panda_hand ns="$(arg arm_id_2)" rpy="0 0 ${-pi/4}" connected_to="$(arg arm_id_2)_link8"/>
     </xacro:if>
+    <xacro:if value="${hand_2 == 'panda_hand_no_gamma'}">
+        <xacro:panda_hand ns="$(arg arm_id_2)" rpy="0 0 ${-pi/4}" connected_to="$(arg arm_id_2)_link8" link="no_gamma"/>
+    </xacro:if>
     <xacro:if value="${hand_2 == 'panda_gelslim'}">
         <xacro:panda_gelslim ns="$(arg arm_id_2)" rpy="0 0 ${-pi/4}" connected_to="$(arg arm_id_2)_link8"/>

File: mmint_franka_moveit_config/config/panda.srdf.xacro (robot description, xacro)
@@ -17,5 +17,5 @@
     <!--SUBGROUPS: Groups can also be formed by referencing to already defined group names-->
     <!--  Depending on selected hands, setup the kinematic chain accordingly.  -->
-    <xacro:if value="${hand_1 == 'panda_hand' or hand_1 == 'panda_gelslim'}">
+    <xacro:if value="${hand_1 == 'panda_hand' or hand_1 == 'panda_hand_no_gamma' or hand_1 == 'panda_gelslim'}">
         <group name="$(arg arm_id_1)">
             <chain base_link="$(arg arm_id_1)_link0" tip_link="$(arg arm_id_1)_gripper_origin"/>
@@ -33,10 +33,10 @@
     </xacro:if>
     <xacro:unless
-            value="${hand_1 == 'panda_hand' or hand_1 == 'panda_gelslim' or hand_1 == 'gamma' or hand_1 == 'sponge_eef' or hand_1 == 'sponge_eef_extend'}">
+            value="${hand_1 == 'panda_hand' or hand_1 == 'panda_hand_no_gamma' or hand_1 == 'panda_gelslim' or hand_1 == 'gamma' or hand_1 == 'sponge_eef' or hand_1 == 'sponge_eef_extend'}">
         <group name="$(arg arm_id_1)">
             <chain base_link="$(arg arm_id_1)_link0" tip_link="$(arg arm_id_1)_link8"/>
         </group>
     </xacro:unless>
-    <xacro:if value="${hand_2 == 'panda_hand' or hand_2 == 'panda_gelslim'}">
+    <xacro:if value="${hand_2 == 'panda_hand' or hand_2 == 'panda_hand_no_gamma' or hand_2 == 'panda_gelslim'}">
         <group name="$(arg arm_id_2)">
             <chain base_link="$(arg arm_id_2)_link0" tip_link="$(arg arm_id_2)_gripper_origin"/>
@@ -54,5 +54,5 @@
     </xacro:if>
     <xacro:unless
-            value="${hand_2 == 'panda_hand' or hand_2 == 'panda_gelslim' or hand_2 == 'gamma' or hand_1 == 'sponge_eef' or hand_1 == 'sponge_eef_extend'}">
+            value="${hand_2 == 'panda_hand' or hand_2 == 'panda_hand_no_gamma' or hand_2 == 'panda_gelslim' or hand_2 == 'gamma' or hand_1 == 'sponge_eef' or hand_1 == 'sponge_eef_extend'}">
         <group name="$(arg arm_id_2)">
             <chain base_link="$(arg arm_id_2)_link0" tip_link="$(arg arm_id_2)_link8"/>
@@ -157,4 +157,10 @@
         <disable_collisions link1="$(arg arm_id_1)_leftfinger" link2="$(arg arm_id_1)_rightfinger" reason="Default"/>
     </xacro:if>
+    <xacro:if value="${hand_1 == 'panda_hand_no_gamma'}">
+        <disable_collisions link1="$(arg arm_id_1)_hand" link2="$(arg arm_id_1)_link7_sc" reason="Adjacent"/>
+        <disable_collisions link1="$(arg arm_id_1)_hand" link2="$(arg arm_id_1)_leftfinger" reason="Adjacent"/>
+        <disable_collisions link1="$(arg arm_id_1)_hand" link2="$(arg arm_id_1)_rightfinger" reason="Adjacent"/>
+        <disable_collisions link1="$(arg arm_id_1)_leftfinger" link2="$(arg arm_id_1)_rightfinger" reason="Default"/>
+    </xacro:if>
     <xacro:if value="${hand_1 == 'gamma'}">
         <disable_collisions link1="$(arg arm_id_1)_ft" link2="$(arg arm_id_1)_link7_sc" reason="Adjacent"/>
@@ -176,4 +182,10 @@
         <disable_collisions link1="$(arg arm_id_2)_leftfinger" link2="$(arg arm_id_2)_rightfinger" reason="Default"/>
     </xacro:if>
+    <xacro:if value="${hand_2 == 'panda_hand_no_gamma'}">
+        <disable_collisions link1="$(arg arm_id_2)_hand" link2="$(arg arm_id_2)_link7_sc" reason="Adjacent"/>
+        <disable_collisions link1="$(arg arm_id_2)_hand" link2="$(arg arm_id_2)_leftfinger" reason="Adjacent"/>
+        <disable_collisions link1="$(arg arm_id_2)_hand" link2="$(arg arm_id_2)_rightfinger" reason="Adjacent"/>
+        <disable_collisions link1="$(arg arm_id_2)_leftfinger" link2="$(arg arm_id_2)_rightfinger" reason="Default"/>
+    </xacro:if>
     <xacro:if value="${hand_2 == 'gamma'}">
         <disable_collisions link1="$(arg arm_id_2)_ft" link2="$(arg arm_id_2)_link7_sc" reason="Adjacent"/>

Commit message: adding some mess to make the panda moveit work without sponge and no ft sensor

File: mmint_franka_description/robots/hands/panda_hand.xacro (robot description, xacro)
@@ -3,5 +3,5 @@
     <xacro:include filename="$(find mmint_franka_description)/robots/hands/gamma.xacro"/>
     <xacro:macro name="panda_hand" params="connected_to:='' ns:='' rpy:='0 0 0' xyz:='0 0 0' link:='gamma'">
-        <xacro:if value="${link == 'gamma'}">
+        <!-- <xacro:if value="${link == 'gamma'}">
             <xacro:gamma ns="${ns}" connected_to="${connected_to}" rpy="${rpy}" xyz="${xyz}"/>
             <joint name="${ns}_hand_joint" type="fixed">
@@ -10,6 +10,6 @@
                 <origin xyz="0 0 0.0079" rpy="0 0 0"/>
             </joint>
-        </xacro:if>
-        <xacro:unless value="${link == 'gamma'}">
+        </xacro:if> -->
+        <!-- <xacro:unless value="${link == 'gamma'}">
             <joint name="${ns}_hand_joint" type="fixed">
                 <parent link="${connected_to}"/>
@@ -17,6 +17,11 @@
                 <origin xyz="${xyz}" rpy="${rpy}"/>
             </joint>
-        </xacro:unless>
+        </xacro:unless> -->
         <!--        <xacro:gamma ns="${ns}" connected_to="${connected_to}" rpy="${rpy}" xyz="${xyz}"/>-->
+        <joint name="${ns}_hand_joint" type="fixed">
+                <parent link="${connected_to}"/>
+                <child link="${ns}_hand"/>
+                <origin xyz="${xyz}" rpy="${rpy}"/>
+            </joint>
         <link name="${ns}_hand">
             <visual>

File: mmint_franka_description/robots/mmint_panda.urdf.xacro (robot description, xacro)
@@ -2,5 +2,5 @@
 <robot xmlns:xacro="http://www.ros.org/wiki/xacro" name="panda">
     <xacro:arg name="arm_id" default="panda_1"/>
-    <xacro:arg name="hand" default="panda_hand"/>
+    <xacro:arg name="hand" default="panda_hand_no_gamma"/>
     <xacro:arg name="arm_xyz_base" default="0 0.4425 0.6"/>
     <xacro:arg name="arm_rpy_base" default="0.0 0.0 -1.57079633"/>

File: mmint_franka_single_moveit_config/config/panda.srdf.xacro (robot description, xacro)
@@ -6,5 +6,5 @@
 <robot xmlns:xacro="http://www.ros.org/wiki/xacro" name="panda">
     <xacro:arg name="arm_id" default="panda_1"/>
-    <xacro:arg name="hand" default="panda_hand"/>
+    <xacro:arg name="hand" default="panda_hand_no_gamma"/>
     <xacro:property name="hand" value="$(arg hand)"/>
     <!--GROUPS: Representation of a set of joints and links. This can be useful for specifying DOF to plan for, defining arms, end effectors, etc-->
@@ -14,5 +14,5 @@
     <!--SUBGROUPS: Groups can also be formed by referencing to already defined group names-->
     <group name="$(arg arm_id)">
-        <chain base_link="$(arg arm_id)_link0" tip_link="$(arg arm_id)_mount"/>
+        <chain base_link="$(arg arm_id)_link0" tip_link="$(arg arm_id)_link8"/>
     </group>
     <!--  Define some useful group positions  -->
@@ -73,5 +73,19 @@
     <xacro:configure_collisions arm_id="$(arg arm_id)" link="6"/>
     <xacro:configure_collisions arm_id="$(arg arm_id)" link="7"/>
-    <xacro:if value="${hand == 'sponge_eef_extend_no_gamma'}">
+    <!-- <disable_collisions link1="$(arg arm_id)_hand" link2="$(arg arm_id)_ft" reason="Adjacent"/> -->
+    <!-- <disable_collisions link1="$(arg arm_id)_ft" link2="$(arg arm_id)_link7_sc" reason="Adjacent"/> -->
+    <disable_collisions link1="$(arg arm_id)_hand" link2="$(arg arm_id)_link7_sc" reason="Adjacent"/>
+    <disable_collisions link1="$(arg arm_id)_hand" link2="$(arg arm_id)_leftfinger" reason="Adjacent"/>
+    <disable_collisions link1="$(arg arm_id)_hand" link2="$(arg arm_id)_rightfinger" reason="Adjacent"/>
+    <disable_collisions link1="$(arg arm_id)_leftfinger" link2="$(arg arm_id)_rightfinger" reason="Default"/>
+<!--
+    <xacro:if value="${hand == 'panda_hand' or hand == 'panda_gelslim'}">
+        <disable_collisions link1="$(arg arm_id)_hand" link2="$(arg arm_id)_ft" reason="Adjacent"/>
+        <disable_collisions link1="$(arg arm_id)_ft" link2="$(arg arm_id)_link7_sc" reason="Adjacent"/>
+        <disable_collisions link1="$(arg arm_id)_hand" link2="$(arg arm_id)_leftfinger" reason="Adjacent"/>
+        <disable_collisions link1="$(arg arm_id)_hand" link2="$(arg arm_id)_rightfinger" reason="Adjacent"/>
+        <disable_collisions link1="$(arg arm_id)_leftfinger" link2="$(arg arm_id)_rightfinger" reason="Default"/>
+    </xacro:if> -->
+    <!-- <xacro:if value="${hand == 'sponge_eef_extend_no_gamma'}">
         <disable_collisions link1="$(arg arm_id)_ft" link2="$(arg arm_id)_link7_sc" reason="Adjacent"/>
         <disable_collisions link1="$(arg arm_id)_ft" link2="$(arg arm_id)_mount_extend" reason="Adjacent"/>
@@ -81,4 +95,4 @@
         <disable_collisions link1="$(arg arm_id)_ft" link2="$(arg arm_id)_link7_sc" reason="Adjacent"/>
         <disable_collisions link1="$(arg arm_id)_ft" link2="$(arg arm_id)_mount" reason="Adjacent"/>
-    </xacro:if>
+    </xacro:if> -->
 </robot>
