Commit message: Add new wrist camera attachment and better args for xacro setup

File: mmint_franka_description/robots/hands/panda_gelsight.xacro (robot description, xacro)
@@ -2,20 +2,10 @@
 <robot xmlns:xacro="http://www.ros.org/wiki/xacro" name="panda_gelslim">
     <xacro:include filename="$(find mmint_franka_description)/robots/hands/gamma.xacro"/>
-    <xacro:macro name="panda_gelsight" params="connected_to:='' ns:='' rpy:='0 0 0' xyz:='0 0 0' link:=''">
-        <xacro:if value="${link == 'gamma'}">
-            <xacro:gamma ns="${ns}" connected_to="${connected_to}" rpy="${rpy}" xyz="${xyz}"/>
-            <joint name="${ns}_hand_joint" type="fixed">
-                <parent link="${ns}_ft_origin"/>
-                <child link="${ns}_hand"/>
-                <origin xyz="0 0 0.0079" rpy="0 0 0"/>
-            </joint>
-        </xacro:if>
-        <xacro:unless value="${link == 'gamma'}">
-            <joint name="${ns}_hand_joint" type="fixed">
-                <parent link="${connected_to}"/>
-                <child link="${ns}_hand"/>
-                <origin xyz="${xyz}" rpy="${rpy}"/>
-            </joint>
-        </xacro:unless>
+    <xacro:macro name="panda_gelsight" params="connected_to:='' ns:='' rpy:='0 0 0' xyz:='0 0 0'">
+        <joint name="${ns}_hand_joint" type="fixed">
+            <parent link="${connected_to}"/>
+            <child link="${ns}_hand"/>
+            <origin xyz="${xyz}" rpy="${rpy}"/>
+        </joint>
         <link name="${ns}_hand">
             <visual>

File: mmint_franka_description/robots/hands/panda_hand.xacro (robot description, xacro)
@@ -3,20 +3,9 @@
     <xacro:include filename="$(find mmint_franka_description)/robots/hands/gamma.xacro"/>
     <xacro:macro name="panda_hand" params="connected_to:='' ns:='' rpy:='0 0 0' xyz:='0 0 0' link:='gamma'">
-        <xacro:if value="${link == 'gamma'}">
-            <xacro:gamma ns="${ns}" connected_to="${connected_to}" rpy="${rpy}" xyz="${xyz}"/>
-            <joint name="${ns}_hand_joint" type="fixed">
-                <parent link="${ns}_ft_origin"/>
-                <child link="${ns}_hand"/>
-                <origin xyz="0 0 0.0079" rpy="0 0 0"/>
-            </joint>
-        </xacro:if>
-        <xacro:unless value="${link == 'gamma'}">
-            <joint name="${ns}_hand_joint" type="fixed">
-                <parent link="${connected_to}"/>
-                <child link="${ns}_hand"/>
-                <origin xyz="${xyz}" rpy="${rpy}"/>
-            </joint>
-        </xacro:unless>
-        <!--        <xacro:gamma ns="${ns}" connected_to="${connected_to}" rpy="${rpy}" xyz="${xyz}"/>-->
+        <joint name="${ns}_hand_joint" type="fixed">
+            <parent link="${connected_to}"/>
+            <child link="${ns}_hand"/>
+            <origin xyz="${xyz}" rpy="${rpy}"/>
+        </joint>
         <link name="${ns}_hand">
             <visual>

File: mmint_franka_description/robots/mmint_panda.urdf.xacro (robot description, xacro)
@@ -3,11 +3,16 @@
     <xacro:arg name="arm_id" default="panda_1"/>
     <xacro:arg name="hand" default="panda_hand"/>
+    <xacro:arg name="include_gamma" default="false"/>
+    <xacro:arg name="include_wrist_camera" default="false"/>
     <xacro:arg name="arm_xyz_base" default="0 0.4425 0.6"/>
     <xacro:arg name="arm_rpy_base" default="0.0 0.0 -1.57079633"/>
     <xacro:property name="hand" value="$(arg hand)"/>
+    <xacro:property name="include_gamma" value="$(arg include_gamma)"/>
+    <xacro:property name="include_wrist_camera" value="$(arg include_wrist_camera)"/>
     <!-- Load source xacros -->
     <xacro:include filename="$(find mmint_franka_description)/robots/materials.xacro"/>
     <xacro:include filename="$(find franka_description)/robots/common/franka_arm.xacro"/>
     <xacro:include filename="$(find mmint_franka_description)/robots/hands/gamma.xacro"/>
+    <xacro:include filename="$(find mmint_franka_description)/robots/hands/wrist_camera.xacro"/>
     <xacro:include filename="$(find mmint_franka_description)/robots/hands/panda_hand.xacro"/>
     <xacro:include filename="$(find mmint_franka_description)/robots/hands/panda_gelslim.xacro"/>
@@ -39,37 +44,53 @@
     <xacro:franka_arm arm_id="$(arg arm_id)" connected_to="base" xyz="$(arg arm_xyz_base)" rpy="$(arg arm_rpy_base)"
                       joint_limits="${xacro.load_yaml('$(find franka_description)/robots/panda/joint_limits.yaml')}"/>
+    <link name="$(arg arm_id)_flange"/>
+    <joint name="$(arg arm_id)_flange_joint" type="fixed">
+        <parent link="$(arg arm_id)_link8"/>
+        <child link="$(arg arm_id)_flange"/>
+        <origin rpy="0 0 ${-pi/4}"/>
+    </joint>
+    <xacro:property name="connecting_link" value="$(arg arm_id)_flange"/>
+    <xacro:if value="${include_gamma}">
+        <xacro:gamma ns="$(arg arm_id)" connected_to="$(arg arm_id)_flange"/>
+        <xacro:property name="connecting_link" value="$(arg arm_id)_ft_origin"/>
+    </xacro:if>
+    <xacro:if value="${include_wrist_camera}">
+        <xacro:if value="${include_gamma}">
+            <xacro:wrist_camera ns="$(arg arm_id)" connected_to="$(arg arm_id)_ft_origin"/>
+        </xacro:if>
+        <xacro:unless value="${include_gamma}">
+            <xacro:wrist_camera ns="$(arg arm_id)" connected_to="$(arg arm_id)_flange"/>
+        </xacro:unless>
+        <xacro:property name="connecting_link" value="$(arg arm_id)_wrist_camera_flange"/>
+    </xacro:if>
     <xacro:if value="${hand == 'panda_hand'}">
-        <xacro:panda_hand ns="$(arg arm_id)" rpy="0 0 ${-pi/4}" connected_to="$(arg arm_id)_link8"/>
-    </xacro:if>
-    <xacro:if value="${hand == 'panda_hand_no_gamma'}">
-        <xacro:panda_hand ns="$(arg arm_id)" rpy="0 0 ${-pi/4}" connected_to="$(arg arm_id)_link8" link="no_gamma"/>
+        <xacro:if value="${include_gamma}">
+            <xacro:panda_hand ns="$(arg arm_id)" xyz="0 0 0.0079" connected_to="${connecting_link}"/>
+        </xacro:if>
+        <xacro:unless value="${include_gamma}">
+            <xacro:panda_hand ns="$(arg arm_id)" connected_to="${connecting_link}"/>
+        </xacro:unless>
     </xacro:if>
     <xacro:if value="${hand == 'panda_gelslim'}">
-        <xacro:panda_gelslim ns="$(arg arm_id)" rpy="0 0 ${-pi/4}" connected_to="$(arg arm_id)_link8"/>
-    </xacro:if>
-    <xacro:if value="${hand == 'gamma'}">
-        <xacro:gamma ns="$(arg arm_id)" rpy="0 0 ${-pi/4}" connected_to="$(arg arm_id)_link8"/>
+        <xacro:if value="${include_gamma}">
+            <xacro:panda_gelslim ns="$(arg arm_id)" xyz="0 0 0.0079" connected_to="${connecting_link}"/>
+        </xacro:if>
+        <xacro:unless value="${include_gamma}">
+            <xacro:panda_gelslim ns="$(arg arm_id)" connected_to="${connecting_link}"/>
+        </xacro:unless>
     </xacro:if>
     <xacro:if value="${hand == 'sponge_eef'}">
-        <xacro:sponge_eef ns="$(arg arm_id)" rpy="0 0 ${-pi/4}" connected_to="$(arg arm_id)_link8"
-                          extend="${False}"/>
-    </xacro:if>
-    <xacro:if value="${hand == 'sponge_eef_no_gamma'}">
-        <xacro:sponge_eef ns="$(arg arm_id)" rpy="0 0 ${-pi/4}" connected_to="$(arg arm_id)_link8" extend="${False}"
-                          gamma_="${False}"/>
+        <xacro:sponge_eef ns="$(arg arm_id)" connected_to="${connecting_link}" extend="${False}"/>
     </xacro:if>
     <xacro:if value="${hand == 'sponge_eef_extend'}">
-        <xacro:sponge_eef ns="$(arg arm_id)" rpy="0 0 ${-pi/4}" connected_to="$(arg arm_id)_link8"
-                          extend="${True}"/>
-    </xacro:if>
-    <xacro:if value="${hand == 'sponge_eef_extend_no_gamma'}">
-        <xacro:sponge_eef ns="$(arg arm_id)" rpy="0 0 ${-pi/4}" connected_to="$(arg arm_id)_link8" extend="${True}"
-                          gamma_="${False}"/>
+        <xacro:sponge_eef ns="$(arg arm_id)" connected_to="${connecting_link}" extend="${True}"/>
     </xacro:if>
     <xacro:if value="${hand == 'panda_gelsight'}">
-        <xacro:panda_gelsight ns="$(arg arm_id)" rpy="0 0 ${-pi/4}" connected_to="$(arg arm_id)_link8" link="gamma"/>
-    </xacro:if>
-    <xacro:if value="${hand == 'panda_gelsight_no_gamma'}">
-        <xacro:panda_gelsight ns="$(arg arm_id)" rpy="0 0 ${-pi/4}" connected_to="$(arg arm_id)_link8"/>
+        <xacro:if value="${include_gamma}">
+            <xacro:panda_gelsight ns="$(arg arm_id)" xyz="0 0 0.0079" connected_to="${connecting_link}"/>
+        </xacro:if>
+        <xacro:unless value="${include_gamma}">
+            <xacro:panda_gelsight ns="$(arg arm_id)" connected_to="${connecting_link}"/>
+        </xacro:unless>
     </xacro:if>
 </robot>

Commit message: Update planning scene/urdf with (optional) inserts

File: mmint_franka_description/robots/hands/panda_gelsight.xacro (robot description, xacro)
@@ -2,5 +2,5 @@
 <robot xmlns:xacro="http://www.ros.org/wiki/xacro" name="panda_gelslim">
     <xacro:include filename="$(find mmint_franka_description)/robots/hands/gamma.xacro"/>
-    <xacro:macro name="panda_gelsight" params="connected_to:='' ns:='' rpy:='0 0 0' xyz:='0 0 0'">
+    <xacro:macro name="panda_gelsight" params="connected_to:='' ns:='' rpy:='0 0 0' xyz:='0 0 0' insert:='false'">
         <joint name="${ns}_hand_joint" type="fixed">
             <parent link="${connected_to}"/>
@@ -61,10 +61,20 @@
             </collision>
         </link>
-        <joint name="${ns}_fingerbox_left_joint" type="fixed">
-            <origin rpy="0 0 0" xyz="0.0 0.0 0.0"/>
-            <parent link="${ns}_leftfinger"/>
-            <child link="${ns}_fingerbox_left"/>
-            <axis xyz="0 0 0"/>
-        </joint>
+        <xacro:if value="${insert}">
+            <joint name="${ns}_fingerbox_left_joint" type="fixed">
+                <origin rpy="0 0 0" xyz="0.0 0.0 -0.0054"/>
+                <parent link="${ns}_leftfinger"/>
+                <child link="${ns}_fingerbox_left"/>
+                <axis xyz="0 0 0"/>
+            </joint>
+        </xacro:if>
+        <xacro:unless value="${insert}">
+            <joint name="${ns}_fingerbox_left_joint" type="fixed">
+                <origin rpy="0 0 0" xyz="0.0 0.0 0.0"/>
+                <parent link="${ns}_leftfinger"/>
+                <child link="${ns}_fingerbox_left"/>
+                <axis xyz="0 0 0"/>
+            </joint>
+        </xacro:unless>
         <link name="${ns}_fingerbox_left">
             <visual>
@@ -79,10 +89,20 @@
             </collision>
         </link>
-        <joint name="elastomer_joint_left" type="fixed">
-            <origin rpy="0 0 0" xyz="0.0 0.0 0.0"/>
-            <parent link="${ns}_fingerbox_left"/>
-            <child link="elastomer_left"/>
-            <axis xyz="0 0 0"/>
-        </joint>
+        <xacro:if value="${insert}">
+            <joint name="elastomer_joint_left" type="fixed">
+                <origin rpy="0 0 0" xyz="0.0 0.0 -0.0054"/>
+                <parent link="${ns}_leftfinger"/>
+                <child link="elastomer_left"/>
+                <axis xyz="0 0 0"/>
+            </joint>
+        </xacro:if>
+        <xacro:unless value="${insert}">
+            <joint name="elastomer_joint_left" type="fixed">
+                <origin rpy="0 0 0" xyz="0.0 0.0 0.0"/>
+                <parent link="${ns}_leftfinger"/>
+                <child link="elastomer_left"/>
+                <axis xyz="0 0 0"/>
+            </joint>
+        </xacro:unless>
         <link name="elastomer_left">
             <visual>
@@ -154,10 +174,20 @@
             </collision>
         </link>
-        <joint name="${ns}_fingerbox_right_joint" type="fixed">
-            <origin rpy="0 0 0" xyz="0.0 0.0 0.0"/>
-            <parent link="${ns}_rightfinger"/>
-            <child link="${ns}_fingerbox_right"/>
-            <axis xyz="0 0 0"/>
-        </joint>
+        <xacro:if value="${insert}">
+            <joint name="${ns}_fingerbox_right_joint" type="fixed">
+                <origin rpy="0 0 0" xyz="0.0 0.0 -0.0054"/>
+                <parent link="${ns}_rightfinger"/>
+                <child link="${ns}_fingerbox_right"/>
+                <axis xyz="0 0 0"/>
+            </joint>
+        </xacro:if>
+        <xacro:unless value="${insert}">
+            <joint name="${ns}_fingerbox_right_joint" type="fixed">
+                <origin rpy="0 0 0" xyz="0.0 0.0 0.0"/>
+                <parent link="${ns}_rightfinger"/>
+                <child link="${ns}_fingerbox_right"/>
+                <axis xyz="0 0 0"/>
+            </joint>
+        </xacro:unless>
         <link name="${ns}_fingerbox_right">
             <visual>
@@ -172,10 +202,20 @@
             </collision>
         </link>
-        <joint name="elastomer_joint_right" type="fixed">
-            <origin rpy="0 0 0" xyz="0.0 0.0 0.0"/>
-            <parent link="${ns}_rightfinger"/>
-            <child link="elastomer_right"/>
-            <axis xyz="0 0 0"/>
-        </joint>
+        <xacro:if value="${insert}">
+            <joint name="elastomer_joint_right" type="fixed">
+                <origin rpy="0 0 0" xyz="0.0 0.0 -0.0054"/>
+                <parent link="${ns}_rightfinger"/>
+                <child link="elastomer_right"/>
+                <axis xyz="0 0 0"/>
+            </joint>
+        </xacro:if>
+        <xacro:unless value="${insert}">
+            <joint name="elastomer_joint_right" type="fixed">
+                <origin rpy="0 0 0" xyz="0.0 0.0 0.0"/>
+                <parent link="${ns}_rightfinger"/>
+                <child link="elastomer_right"/>
+                <axis xyz="0 0 0"/>
+            </joint>
+        </xacro:unless>
         <link name="elastomer_right">         <!-- surface tip of the elastomer  -->
             <visual>

File: mmint_franka_description/robots/mmint_panda.urdf.xacro (robot description, xacro)
@@ -5,4 +5,5 @@
     <xacro:arg name="include_gamma" default="false"/>
     <xacro:arg name="include_wrist_camera" default="false"/>
+    <xacro:arg name="include_gelsight_inserts" default="false"/>
     <xacro:arg name="arm_xyz_base" default="0 0.4425 0.6"/>
     <xacro:arg name="arm_rpy_base" default="0.0 0.0 -1.57079633"/>
@@ -10,4 +11,5 @@
     <xacro:property name="include_gamma" value="$(arg include_gamma)"/>
     <xacro:property name="include_wrist_camera" value="$(arg include_wrist_camera)"/>
+    <xacro:property name="include_gelsight_inserts" value="$(arg include_gelsight_inserts)"/>
     <!-- Load source xacros -->
     <xacro:include filename="$(find mmint_franka_description)/robots/materials.xacro"/>
@@ -89,12 +91,15 @@
         <xacro:if value="${include_gamma}">
             <xacro:if value="${include_wrist_camera}">
-                <xacro:panda_gelsight ns="$(arg arm_id)" connected_to="${connecting_link}"/>
+                <xacro:panda_gelsight ns="$(arg arm_id)" connected_to="${connecting_link}"
+                                      insert="${include_gelsight_inserts}"/>
             </xacro:if>
             <xacro:unless value="${include_wrist_camera}">
-                <xacro:panda_gelsight ns="$(arg arm_id)" xyz="0 0 0.0079" connected_to="${connecting_link}"/>
+                <xacro:panda_gelsight ns="$(arg arm_id)" xyz="0 0 0.0079" connected_to="${connecting_link}"
+                                      insert="${include_gelsight_inserts}"/>
             </xacro:unless>
         </xacro:if>
         <xacro:unless value="${include_gamma}">
-            <xacro:panda_gelsight ns="$(arg arm_id)" connected_to="${connecting_link}"/>
+            <xacro:panda_gelsight ns="$(arg arm_id)" connected_to="${connecting_link}"
+                                  insert="${include_gelsight_inserts}"/>
         </xacro:unless>
     </xacro:if>

File: mmint_franka_single_moveit_config/config/panda.srdf.xacro (robot description, xacro)
@@ -77,4 +77,8 @@
     <xacro:configure_collisions arm_id="$(arg arm_id)" link="6"/>
     <xacro:configure_collisions arm_id="$(arg arm_id)" link="7"/>
+    <xacro:if value="${include_gamma}">
+        <xacro:disable_collisions_for link="$(arg arm_id)_ft"
+                                      others="${['$(arg arm_id)_link7', '$(arg arm_id)_link7_sc', '$(arg arm_id)_link8']}"/>
+    </xacro:if>
     <xacro:if value="${hand == 'panda_gelsight'}">
         <xacro:if value="${include_gamma}">
