Commit message: Make srdf xacro and add args to switch EE

File: mmint_franka_moveit_config/config/panda.srdf.xacro (robot description, xacro)
@@ -4,5 +4,11 @@
     A URDF file must exist for this robot as well, where the joints and the links that are referenced are defined
 -->
-<robot name="panda">
+<robot xmlns:xacro="http://www.ros.org/wiki/xacro" name="panda">
+    <xacro:arg name="arm_id_1" default="panda_1"/>
+    <xacro:arg name="arm_id_2" default="panda_2"/>
+    <xacro:arg name="hand_1" default="panda_hand"/>
+    <xacro:arg name="hand_2" default="panda_hand"/>
+    <xacro:property name="hand_1" value="$(arg hand_1)"/>
+    <xacro:property name="hand_2" value="$(arg hand_2)"/>
     <!--GROUPS: Representation of a set of joints and links. This can be useful for specifying DOF to plan for, defining arms, end effectors, etc-->
     <!--LINKS: When a link is specified, the parent joint of that link (if it exists) is automatically included-->
@@ -29,4 +35,57 @@
     </group>
     <!--DISABLE COLLISIONS: By default it is assumed that any link of the robot could potentially come into collision with any other link in the robot. This tag disables collision checking between a specified pair of links. -->
+    <!-- Disable collisions for each hand type -->
+    <xacro:if value="${hand_1 == 'panda_hand' or hand_1 == 'panda_gelslim'}">
+        <disable_collisions link1="$(arg arm_id_1)_hand" link2="$(arg arm_id_1)_ft" reason="Adjacent"/>
+        <disable_collisions link1="$(arg arm_id_1)_ft" link2="$(arg arm_id_1)_link7" reason="Adjacent"/>
+        <disable_collisions link1="$(arg arm_id_1)_ft" link2="$(arg arm_id_1)_link7_sc" reason="Adjacent"/>
+        <disable_collisions link1="$(arg arm_id_1)_hand" link2="$(arg arm_id_1)_leftfinger" reason="Adjacent"/>
+        <disable_collisions link1="$(arg arm_id_1)_hand" link2="$(arg arm_id_1)_rightfinger" reason="Adjacent"/>
+        <disable_collisions link1="$(arg arm_id_1)_leftfinger" link2="$(arg arm_id_1)_link3" reason="Never"/>
+        <disable_collisions link1="$(arg arm_id_1)_leftfinger" link2="$(arg arm_id_1)_link4" reason="Never"/>
+        <disable_collisions link1="$(arg arm_id_1)_leftfinger" link2="$(arg arm_id_1)_link6" reason="Never"/>
+        <disable_collisions link1="$(arg arm_id_1)_leftfinger" link2="$(arg arm_id_1)_link7" reason="Never"/>
+        <disable_collisions link1="$(arg arm_id_1)_leftfinger" link2="$(arg arm_id_1)_rightfinger" reason="Default"/>
+        <disable_collisions link1="$(arg arm_id_1)_link3" link2="$(arg arm_id_1)_rightfinger" reason="Never"/>
+        <disable_collisions link1="$(arg arm_id_1)_link4" link2="$(arg arm_id_1)_rightfinger" reason="Never"/>
+        <disable_collisions link1="$(arg arm_id_1)_link6" link2="$(arg arm_id_1)_rightfinger" reason="Never"/>
+        <disable_collisions link1="$(arg arm_id_1)_link7" link2="$(arg arm_id_1)_rightfinger" reason="Never"/>
+        <disable_collisions link1="$(arg arm_id_1)_hand" link2="$(arg arm_id_1)_link3" reason="Never"/>
+        <disable_collisions link1="$(arg arm_id_1)_hand" link2="$(arg arm_id_1)_link4" reason="Never"/>
+        <disable_collisions link1="$(arg arm_id_1)_hand" link2="$(arg arm_id_1)_link6" reason="Never"/>
+        <disable_collisions link1="$(arg arm_id_1)_hand" link2="$(arg arm_id_1)_link7" reason="Adjacent"/>
+    </xacro:if>
+    <xacro:if value="${hand_1 == 'panda_ft'}">
+        <disable_collisions link1="$(arg arm_id_1)_link3" link2="$(arg arm_id_1)_link_ft" reason="Never"/>
+        <disable_collisions link1="$(arg arm_id_1)_link4" link2="$(arg arm_id_1)_link_ft" reason="Never"/>
+        <disable_collisions link1="$(arg arm_id_1)_link6" link2="$(arg arm_id_1)_link_ft" reason="Never"/>
+        <disable_collisions link1="$(arg arm_id_1)_link7" link2="$(arg arm_id_1)_link_ft" reason="Never"/>
+    </xacro:if>
+    <xacro:if value="${hand_2 == 'panda_hand' or hand_2 == 'panda_gelslim'}">
+        <disable_collisions link1="$(arg arm_id_2)_hand" link2="$(arg arm_id_2)_ft" reason="Adjacent"/>
+        <disable_collisions link1="$(arg arm_id_2)_ft" link2="$(arg arm_id_2)_link7" reason="Adjacent"/>
+        <disable_collisions link1="$(arg arm_id_2)_ft" link2="$(arg arm_id_2)_link7_sc" reason="Adjacent"/>
+        <disable_collisions link1="$(arg arm_id_2)_hand" link2="$(arg arm_id_2)_leftfinger" reason="Adjacent"/>
+        <disable_collisions link1="$(arg arm_id_2)_hand" link2="$(arg arm_id_2)_rightfinger" reason="Adjacent"/>
+        <disable_collisions link1="$(arg arm_id_2)_leftfinger" link2="$(arg arm_id_2)_link3" reason="Never"/>
+        <disable_collisions link1="$(arg arm_id_2)_leftfinger" link2="$(arg arm_id_2)_link4" reason="Never"/>
+        <disable_collisions link1="$(arg arm_id_2)_leftfinger" link2="$(arg arm_id_2)_link6" reason="Never"/>
+        <disable_collisions link1="$(arg arm_id_2)_leftfinger" link2="$(arg arm_id_2)_link7" reason="Never"/>
+        <disable_collisions link1="$(arg arm_id_2)_leftfinger" link2="$(arg arm_id_2)_rightfinger" reason="Default"/>
+        <disable_collisions link1="$(arg arm_id_2)_link3" link2="$(arg arm_id_2)_rightfinger" reason="Never"/>
+        <disable_collisions link1="$(arg arm_id_2)_link4" link2="$(arg arm_id_2)_rightfinger" reason="Never"/>
+        <disable_collisions link1="$(arg arm_id_2)_link6" link2="$(arg arm_id_2)_rightfinger" reason="Never"/>
+        <disable_collisions link1="$(arg arm_id_2)_link7" link2="$(arg arm_id_2)_rightfinger" reason="Never"/>
+        <disable_collisions link1="$(arg arm_id_2)_hand" link2="$(arg arm_id_2)_link3" reason="Never"/>
+        <disable_collisions link1="$(arg arm_id_2)_hand" link2="$(arg arm_id_2)_link4" reason="Never"/>
+        <disable_collisions link1="$(arg arm_id_2)_hand" link2="$(arg arm_id_2)_link6" reason="Never"/>
+        <disable_collisions link1="$(arg arm_id_2)_hand" link2="$(arg arm_id_2)_link7" reason="Adjacent"/>
+    </xacro:if>
+    <xacro:if value="${hand_2 == 'panda_ft'}">
+        <disable_collisions link1="$(arg arm_id_2)_link3" link2="$(arg arm_id_2)_link_ft" reason="Never"/>
+        <disable_collisions link1="$(arg arm_id_2)_link4" link2="$(arg arm_id_2)_link_ft" reason="Never"/>
+        <disable_collisions link1="$(arg arm_id_2)_link6" link2="$(arg arm_id_2)_link_ft" reason="Never"/>
+        <disable_collisions link1="$(arg arm_id_2)_link7" link2="$(arg arm_id_2)_link_ft" reason="Never"/>
+    </xacro:if>
     <disable_collisions link1="base" link2="panda_1_link0" reason="Adjacent"/>
     <disable_collisions link1="base" link2="panda_1_link0_sc" reason="Default"/>
@@ -48,31 +107,4 @@
     <disable_collisions link1="base" link2="panda_2_link4" reason="Never"/>
     <disable_collisions link1="base" link2="panda_2_link4_sc" reason="Never"/>
-    <disable_collisions link1="panda_1_ft" link2="panda_1_hand" reason="Adjacent"/>
-    <disable_collisions link1="panda_1_ft" link2="panda_1_leftfinger" reason="Never"/>
-    <disable_collisions link1="panda_1_ft" link2="panda_1_link3" reason="Never"/>
-    <disable_collisions link1="panda_1_ft" link2="panda_1_link4" reason="Never"/>
-    <disable_collisions link1="panda_1_ft" link2="panda_1_link4_sc" reason="Never"/>
-    <disable_collisions link1="panda_1_ft" link2="panda_1_link5_sc" reason="Never"/>
-    <disable_collisions link1="panda_1_ft" link2="panda_1_link6" reason="Never"/>
-    <disable_collisions link1="panda_1_ft" link2="panda_1_link6_sc" reason="Never"/>
-    <disable_collisions link1="panda_1_ft" link2="panda_1_link7" reason="Adjacent"/>
-    <disable_collisions link1="panda_1_ft" link2="panda_1_link7_sc" reason="Default"/>
-    <disable_collisions link1="panda_1_ft" link2="panda_1_rightfinger" reason="Never"/>
-    <disable_collisions link1="panda_1_hand" link2="panda_1_leftfinger" reason="Adjacent"/>
-    <disable_collisions link1="panda_1_hand" link2="panda_1_link3" reason="Never"/>
-    <disable_collisions link1="panda_1_hand" link2="panda_1_link4" reason="Never"/>
-    <disable_collisions link1="panda_1_hand" link2="panda_1_link4_sc" reason="Never"/>
-    <disable_collisions link1="panda_1_hand" link2="panda_1_link6" reason="Never"/>
-    <disable_collisions link1="panda_1_hand" link2="panda_1_link6_sc" reason="Never"/>
-    <disable_collisions link1="panda_1_hand" link2="panda_1_link7" reason="Never"/>
-    <disable_collisions link1="panda_1_hand" link2="panda_1_link7_sc" reason="Never"/>
-    <disable_collisions link1="panda_1_hand" link2="panda_1_rightfinger" reason="Adjacent"/>
-    <disable_collisions link1="panda_1_leftfinger" link2="panda_1_link3" reason="Never"/>
-    <disable_collisions link1="panda_1_leftfinger" link2="panda_1_link4_sc" reason="Never"/>
-    <disable_collisions link1="panda_1_leftfinger" link2="panda_1_link6" reason="Never"/>
-    <disable_collisions link1="panda_1_leftfinger" link2="panda_1_link6_sc" reason="Never"/>
-    <disable_collisions link1="panda_1_leftfinger" link2="panda_1_link7" reason="Never"/>
-    <disable_collisions link1="panda_1_leftfinger" link2="panda_1_link7_sc" reason="Never"/>
-    <disable_collisions link1="panda_1_leftfinger" link2="panda_1_rightfinger" reason="Never"/>
     <disable_collisions link1="panda_1_link0" link2="panda_1_link0_sc" reason="Adjacent"/>
     <disable_collisions link1="panda_1_link0" link2="panda_1_link1" reason="Adjacent"/>
@@ -176,5 +208,4 @@
     <disable_collisions link1="panda_1_link3" link2="panda_1_link7" reason="Never"/>
     <disable_collisions link1="panda_1_link3" link2="panda_1_link7_sc" reason="Never"/>
-    <disable_collisions link1="panda_1_link3" link2="panda_1_rightfinger" reason="Never"/>
     <disable_collisions link1="panda_1_link3" link2="panda_2_link0" reason="Never"/>
     <disable_collisions link1="panda_1_link3" link2="panda_2_link0_sc" reason="Never"/>
@@ -211,5 +242,4 @@
     <disable_collisions link1="panda_1_link4_sc" link2="panda_1_link7" reason="Never"/>
     <disable_collisions link1="panda_1_link4_sc" link2="panda_1_link7_sc" reason="Never"/>
-    <disable_collisions link1="panda_1_link4_sc" link2="panda_1_rightfinger" reason="Never"/>
     <disable_collisions link1="panda_1_link4_sc" link2="panda_2_link0" reason="Never"/>
     <disable_collisions link1="panda_1_link4_sc" link2="panda_2_link0_sc" reason="Never"/>
@@ -231,51 +261,15 @@
     <disable_collisions link1="panda_1_link6" link2="panda_1_link7" reason="Adjacent"/>
     <disable_collisions link1="panda_1_link6" link2="panda_1_link7_sc" reason="Default"/>
-    <disable_collisions link1="panda_1_link6" link2="panda_1_rightfinger" reason="Never"/>
-    <disable_collisions link1="panda_1_link6" link2="panda_2_ft" reason="Default"/>
-    <disable_collisions link1="panda_1_link6" link2="panda_2_hand" reason="Default"/>
     <disable_collisions link1="panda_1_link6" link2="panda_2_link5_sc" reason="Default"/>
     <disable_collisions link1="panda_1_link6" link2="panda_2_link7_sc" reason="Default"/>
     <disable_collisions link1="panda_1_link6_sc" link2="panda_1_link7" reason="Never"/>
     <disable_collisions link1="panda_1_link6_sc" link2="panda_1_link7_sc" reason="Default"/>
-    <disable_collisions link1="panda_1_link6_sc" link2="panda_1_rightfinger" reason="Never"/>
     <disable_collisions link1="panda_1_link6_sc" link2="panda_2_link5_sc" reason="Default"/>
     <disable_collisions link1="panda_1_link6_sc" link2="panda_2_link6" reason="Default"/>
     <disable_collisions link1="panda_1_link6_sc" link2="panda_2_link6_sc" reason="Default"/>
     <disable_collisions link1="panda_1_link7" link2="panda_1_link7_sc" reason="Adjacent"/>
-    <disable_collisions link1="panda_1_link7" link2="panda_1_rightfinger" reason="Never"/>
-    <disable_collisions link1="panda_1_link7_sc" link2="panda_1_rightfinger" reason="Never"/>
-    <disable_collisions link1="panda_1_link7_sc" link2="panda_2_ft" reason="Default"/>
-    <disable_collisions link1="panda_1_link7_sc" link2="panda_2_hand" reason="Default"/>
     <disable_collisions link1="panda_1_link7_sc" link2="panda_2_link5" reason="Default"/>
     <disable_collisions link1="panda_1_link7_sc" link2="panda_2_link5_sc" reason="Default"/>
     <disable_collisions link1="panda_1_link7_sc" link2="panda_2_link7_sc" reason="Default"/>
-    <disable_collisions link1="panda_2_ft" link2="panda_2_hand" reason="Adjacent"/>
-    <disable_collisions link1="panda_2_ft" link2="panda_2_leftfinger" reason="Never"/>
-    <disable_collisions link1="panda_2_ft" link2="panda_2_link3" reason="Never"/>
-    <disable_collisions link1="panda_2_ft" link2="panda_2_link4" reason="Never"/>
-    <disable_collisions link1="panda_2_ft" link2="panda_2_link4_sc" reason="Never"/>
-    <disable_collisions link1="panda_2_ft" link2="panda_2_link5_sc" reason="Never"/>
-    <disable_collisions link1="panda_2_ft" link2="panda_2_link6" reason="Never"/>
-    <disable_collisions link1="panda_2_ft" link2="panda_2_link6_sc" reason="Never"/>
-    <disable_collisions link1="panda_2_ft" link2="panda_2_link7" reason="Adjacent"/>
-    <disable_collisions link1="panda_2_ft" link2="panda_2_link7_sc" reason="Default"/>
-    <disable_collisions link1="panda_2_ft" link2="panda_2_rightfinger" reason="Never"/>
-    <disable_collisions link1="panda_2_hand" link2="panda_2_leftfinger" reason="Adjacent"/>
-    <disable_collisions link1="panda_2_hand" link2="panda_2_link3" reason="Never"/>
-    <disable_collisions link1="panda_2_hand" link2="panda_2_link4" reason="Never"/>
-    <disable_collisions link1="panda_2_hand" link2="panda_2_link4_sc" reason="Never"/>
-    <disable_collisions link1="panda_2_hand" link2="panda_2_link5_sc" reason="Default"/>
-    <disable_collisions link1="panda_2_hand" link2="panda_2_link6" reason="Never"/>
-    <disable_collisions link1="panda_2_hand" link2="panda_2_link6_sc" reason="Never"/>
-    <disable_collisions link1="panda_2_hand" link2="panda_2_link7" reason="Never"/>
-    <disable_collisions link1="panda_2_hand" link2="panda_2_link7_sc" reason="Never"/>
-    <disable_collisions link1="panda_2_hand" link2="panda_2_rightfinger" reason="Adjacent"/>
-    <disable_collisions link1="panda_2_leftfinger" link2="panda_2_link3" reason="Never"/>
-    <disable_collisions link1="panda_2_leftfinger" link2="panda_2_link4_sc" reason="Never"/>
-    <disable_collisions link1="panda_2_leftfinger" link2="panda_2_link6" reason="Never"/>
-    <disable_collisions link1="panda_2_leftfinger" link2="panda_2_link6_sc" reason="Never"/>
-    <disable_collisions link1="panda_2_leftfinger" link2="panda_2_link7" reason="Never"/>
-    <disable_collisions link1="panda_2_leftfinger" link2="panda_2_link7_sc" reason="Never"/>
-    <disable_collisions link1="panda_2_leftfinger" link2="panda_2_rightfinger" reason="Default"/>
     <disable_collisions link1="panda_2_link0" link2="panda_2_link0_sc" reason="Adjacent"/>
     <disable_collisions link1="panda_2_link0" link2="panda_2_link1" reason="Adjacent"/>
@@ -325,5 +319,4 @@
     <disable_collisions link1="panda_2_link3" link2="panda_2_link7" reason="Never"/>
     <disable_collisions link1="panda_2_link3" link2="panda_2_link7_sc" reason="Never"/>
-    <disable_collisions link1="panda_2_link3" link2="panda_2_rightfinger" reason="Never"/>
     <disable_collisions link1="panda_2_link3_sc" link2="panda_2_link4" reason="Always"/>
     <disable_collisions link1="panda_2_link3_sc" link2="panda_2_link4_sc" reason="Always"/>
@@ -347,5 +340,4 @@
     <disable_collisions link1="panda_2_link4_sc" link2="panda_2_link7" reason="Never"/>
     <disable_collisions link1="panda_2_link4_sc" link2="panda_2_link7_sc" reason="Never"/>
-    <disable_collisions link1="panda_2_link4_sc" link2="panda_2_rightfinger" reason="Never"/>
     <disable_collisions link1="panda_2_link5" link2="panda_2_link5_sc" reason="Adjacent"/>
     <disable_collisions link1="panda_2_link5" link2="panda_2_link6" reason="Adjacent"/>
@@ -358,10 +350,6 @@
     <disable_collisions link1="panda_2_link6" link2="panda_2_link7" reason="Adjacent"/>
     <disable_collisions link1="panda_2_link6" link2="panda_2_link7_sc" reason="Default"/>
-    <disable_collisions link1="panda_2_link6" link2="panda_2_rightfinger" reason="Never"/>
     <disable_collisions link1="panda_2_link6_sc" link2="panda_2_link7" reason="Never"/>
     <disable_collisions link1="panda_2_link6_sc" link2="panda_2_link7_sc" reason="Default"/>
-    <disable_collisions link1="panda_2_link6_sc" link2="panda_2_rightfinger" reason="Never"/>
     <disable_collisions link1="panda_2_link7" link2="panda_2_link7_sc" reason="Adjacent"/>
-    <disable_collisions link1="panda_2_link7" link2="panda_2_rightfinger" reason="Never"/>
-    <disable_collisions link1="panda_2_link7_sc" link2="panda_2_rightfinger" reason="Never"/>
 </robot>

Commit message: updated kinematic chain in srdf.xacro to plan through gripper_origin for each arm

File: mmint_franka_moveit_config/config/panda.srdf.xacro (robot description, xacro)
@@ -16,21 +16,9 @@
     <!--CHAINS: When a chain is specified, all the links along the chain (including endpoints) are included in the group. Additionally, all the joints that are parents to included links are also included. This means that joints along the chain and the parent joint of the base link are included in the group-->
     <!--SUBGROUPS: Groups can also be formed by referencing to already defined group names-->
-    <group name="panda_1">
-        <joint name="panda_1_joint1"/>
-        <joint name="panda_1_joint2"/>
-        <joint name="panda_1_joint3"/>
-        <joint name="panda_1_joint4"/>
-        <joint name="panda_1_joint5"/>
-        <joint name="panda_1_joint6"/>
-        <joint name="panda_1_joint7"/>
+    <group name="$(arg arm_id_1)">
+        <chain base_link="$(arg arm_id_1)_link0" tip_link="$(arg arm_id_1)_gripper_origin"/>
     </group>
-    <group name="panda_2">
-        <joint name="panda_2_joint1"/>
-        <joint name="panda_2_joint2"/>
-        <joint name="panda_2_joint3"/>
-        <joint name="panda_2_joint4"/>
-        <joint name="panda_2_joint5"/>
-        <joint name="panda_2_joint6"/>
-        <joint name="panda_2_joint7"/>
+    <group name="$(arg arm_id_2)">
+        <chain base_link="$(arg arm_id_2)_link0" tip_link="$(arg arm_id_2)_gripper_origin"/>
     </group>
     <!--DISABLE COLLISIONS: By default it is assumed that any link of the robot could potentially come into collision with any other link in the robot. This tag disables collision checking between a specified pair of links. -->
