Commit message: Cleanup srdf

File: mmint_franka_moveit_config/config/panda.srdf.xacro (robot description, xacro)
@@ -32,5 +32,6 @@
         </group>
     </xacro:if>
-    <xacro:unless value="${hand_1 == 'panda_hand' or hand_1 == 'panda_gelslim' or hand_1 == 'gamma' or hand_1 == 'sponge_eef' or hand_1 == 'sponge_eef_extend'}">
+    <xacro:unless
+            value="${hand_1 == 'panda_hand' or hand_1 == 'panda_gelslim' or hand_1 == 'gamma' or hand_1 == 'sponge_eef' or hand_1 == 'sponge_eef_extend'}">
         <group name="$(arg arm_id_1)">
             <chain base_link="$(arg arm_id_1)_link0" tip_link="$(arg arm_id_1)_link8"/>
@@ -52,5 +53,6 @@
         </group>
     </xacro:if>
-    <xacro:unless value="${hand_2 == 'panda_hand' or hand_2 == 'panda_gelslim' or hand_2 == 'gamma' or hand_1 == 'sponge_eef' or hand_1 == 'sponge_eef_extend'}">
+    <xacro:unless
+            value="${hand_2 == 'panda_hand' or hand_2 == 'panda_gelslim' or hand_2 == 'gamma' or hand_1 == 'sponge_eef' or hand_1 == 'sponge_eef_extend'}">
         <group name="$(arg arm_id_2)">
             <chain base_link="$(arg arm_id_2)_link0" tip_link="$(arg arm_id_2)_link8"/>
@@ -62,36 +64,66 @@
     </group>
     <!--DISABLE COLLISIONS: By default it is assumed that any link of the robot could potentially come into collision with any other link in the robot. This tag disables collision checking between a specified pair of links. -->
+    <xacro:macro name="disable_collisions_for" params="link:=^ others:=^">
+        <xacro:if value="${others}">
+            <xacro:property name="other" value="${others.pop(0)}"/>
+            <disable_collisions link1="${link}" link2="${other}" reason="Never"/>
+            <!-- recursively call -->
+            <xacro:disable_collisions_for/>
+        </xacro:if>
+    </xacro:macro>
+    <xacro:macro name="enable_collisions_for" params="link:=^ others:=^">
+        <xacro:if value="${others}">
+            <xacro:property name="other" value="${others.pop(0)}"/>
+            <enable_collisions link1="${link}" link2="${other}"/>
+            <!-- recursively call -->
+            <xacro:enable_collisions_for/>
+        </xacro:if>
+    </xacro:macro>
+    <xacro:macro name="configure_collisions" params="arm_id other_arm_id link enabled:=${[]}">
+        <!-- Disable collision checking between normal links, as these are handled by "sc" links -->
+        <disable_default_collisions link="${arm_id}_link${link}"/>
+        <!-- Disable all collision checking for ${link}_sc -->
+        <xacro:property name="link_fmt" value="${arm_id}_link{}_sc"/>
+        <xacro:property name="other_link_fmt" value="${other_arm_id}_link{}_sc"/>
+        <xacro:disable_collisions_for link="${link_fmt.format(link)}"
+                                      others="${[link_fmt.format(i) for i in python.range(8)]}"/>
+        <!-- Re-enable collisions checking for selected links -->
+        <xacro:enable_collisions_for link="${link_fmt.format(link)}" others="${[link_fmt.format(i) for i in enabled]}"/>
+        <xacro:enable_collisions_for link="${link_fmt.format(link)}"
+                                     others="${[other_link_fmt.format(i) for i in python.range(8)]}"/>
+    </xacro:macro>
+    <!-- Handle collision settings within each arm -->
+    <xacro:configure_collisions arm_id="panda_1" other_arm_id="panda_2" link="0" enabled="${[5,6,7]}"/>
+    <xacro:configure_collisions arm_id="panda_1" other_arm_id="panda_2" link="1" enabled="${[5,6,7]}"/>
+    <xacro:configure_collisions arm_id="panda_1" other_arm_id="panda_2" link="2" enabled="${[5,6,7]}"/>
+    <xacro:configure_collisions arm_id="panda_1" other_arm_id="panda_2" link="3" enabled="${[7]}"/>
+    <xacro:configure_collisions arm_id="panda_1" other_arm_id="panda_2" link="4"/>
+    <xacro:configure_collisions arm_id="panda_1" other_arm_id="panda_2" link="5"/>
+    <xacro:configure_collisions arm_id="panda_1" other_arm_id="panda_2" link="6"/>
+    <xacro:configure_collisions arm_id="panda_1" other_arm_id="panda_2" link="7"/>
+    <xacro:configure_collisions arm_id="panda_2" other_arm_id="panda_1" link="0" enabled="${[5,6,7]}"/>
+    <xacro:configure_collisions arm_id="panda_2" other_arm_id="panda_1" link="1" enabled="${[5,6,7]}"/>
+    <xacro:configure_collisions arm_id="panda_2" other_arm_id="panda_1" link="2" enabled="${[5,6,7]}"/>
+    <xacro:configure_collisions arm_id="panda_2" other_arm_id="panda_1" link="3" enabled="${[7]}"/>
+    <xacro:configure_collisions arm_id="panda_2" other_arm_id="panda_1" link="4"/>
+    <xacro:configure_collisions arm_id="panda_2" other_arm_id="panda_1" link="5"/>
+    <xacro:configure_collisions arm_id="panda_2" other_arm_id="panda_1" link="6"/>
+    <xacro:configure_collisions arm_id="panda_2" other_arm_id="panda_1" link="7"/>
     <!-- Disable collisions for each hand type -->
     <xacro:if value="${hand_1 == 'panda_hand' or hand_1 == 'panda_gelslim'}">
         <disable_collisions link1="$(arg arm_id_1)_hand" link2="$(arg arm_id_1)_ft" reason="Adjacent"/>
-        <disable_collisions link1="$(arg arm_id_1)_ft" link2="$(arg arm_id_1)_link7" reason="Adjacent"/>
         <disable_collisions link1="$(arg arm_id_1)_ft" link2="$(arg arm_id_1)_link7_sc" reason="Adjacent"/>
         <disable_collisions link1="$(arg arm_id_1)_hand" link2="$(arg arm_id_1)_leftfinger" reason="Adjacent"/>
         <disable_collisions link1="$(arg arm_id_1)_hand" link2="$(arg arm_id_1)_rightfinger" reason="Adjacent"/>
-        <disable_collisions link1="$(arg arm_id_1)_leftfinger" link2="$(arg arm_id_1)_link3" reason="Never"/>
-        <disable_collisions link1="$(arg arm_id_1)_leftfinger" link2="$(arg arm_id_1)_link4" reason="Never"/>
-        <disable_collisions link1="$(arg arm_id_1)_leftfinger" link2="$(arg arm_id_1)_link6" reason="Never"/>
-        <disable_collisions link1="$(arg arm_id_1)_leftfinger" link2="$(arg arm_id_1)_link7" reason="Never"/>
         <disable_collisions link1="$(arg arm_id_1)_leftfinger" link2="$(arg arm_id_1)_rightfinger" reason="Default"/>
-        <disable_collisions link1="$(arg arm_id_1)_link3" link2="$(arg arm_id_1)_rightfinger" reason="Never"/>
-        <disable_collisions link1="$(arg arm_id_1)_link4" link2="$(arg arm_id_1)_rightfinger" reason="Never"/>
-        <disable_collisions link1="$(arg arm_id_1)_link6" link2="$(arg arm_id_1)_rightfinger" reason="Never"/>
-        <disable_collisions link1="$(arg arm_id_1)_link7" link2="$(arg arm_id_1)_rightfinger" reason="Never"/>
-        <disable_collisions link1="$(arg arm_id_1)_hand" link2="$(arg arm_id_1)_link3" reason="Never"/>
-        <disable_collisions link1="$(arg arm_id_1)_hand" link2="$(arg arm_id_1)_link4" reason="Never"/>
-        <disable_collisions link1="$(arg arm_id_1)_hand" link2="$(arg arm_id_1)_link6" reason="Never"/>
-        <disable_collisions link1="$(arg arm_id_1)_hand" link2="$(arg arm_id_1)_link7" reason="Adjacent"/>
     </xacro:if>
     <xacro:if value="${hand_1 == 'gamma'}">
-        <disable_collisions link1="$(arg arm_id_1)_ft" link2="$(arg arm_id_1)_link7" reason="Adjacent"/>
         <disable_collisions link1="$(arg arm_id_1)_ft" link2="$(arg arm_id_1)_link7_sc" reason="Adjacent"/>
     </xacro:if>
     <xacro:if value="${hand_1 == 'sponge_eef'}">
-        <disable_collisions link1="$(arg arm_id_1)_ft" link2="$(arg arm_id_1)_link7" reason="Adjacent"/>
         <disable_collisions link1="$(arg arm_id_1)_ft" link2="$(arg arm_id_1)_link7_sc" reason="Adjacent"/>
         <disable_collisions link1="$(arg arm_id_1)_ft" link2="$(arg arm_id_1)_mount" reason="Adjacent"/>
     </xacro:if>
     <xacro:if value="${hand_1 == 'sponge_eef_extend'}">
-        <disable_collisions link1="$(arg arm_id_1)_ft" link2="$(arg arm_id_1)_link7" reason="Adjacent"/>
         <disable_collisions link1="$(arg arm_id_1)_ft" link2="$(arg arm_id_1)_link7_sc" reason="Adjacent"/>
         <disable_collisions link1="$(arg arm_id_1)_ft" link2="$(arg arm_id_1)_mount_extend" reason="Adjacent"/>
@@ -100,302 +132,21 @@
     <xacro:if value="${hand_2 == 'panda_hand' or hand_2 == 'panda_gelslim'}">
         <disable_collisions link1="$(arg arm_id_2)_hand" link2="$(arg arm_id_2)_ft" reason="Adjacent"/>
-        <disable_collisions link1="$(arg arm_id_2)_ft" link2="$(arg arm_id_2)_link7" reason="Adjacent"/>
         <disable_collisions link1="$(arg arm_id_2)_ft" link2="$(arg arm_id_2)_link7_sc" reason="Adjacent"/>
         <disable_collisions link1="$(arg arm_id_2)_hand" link2="$(arg arm_id_2)_leftfinger" reason="Adjacent"/>
         <disable_collisions link1="$(arg arm_id_2)_hand" link2="$(arg arm_id_2)_rightfinger" reason="Adjacent"/>
-        <disable_collisions link1="$(arg arm_id_2)_leftfinger" link2="$(arg arm_id_2)_link3" reason="Never"/>
-        <disable_collisions link1="$(arg arm_id_2)_leftfinger" link2="$(arg arm_id_2)_link4" reason="Never"/>
-        <disable_collisions link1="$(arg arm_id_2)_leftfinger" link2="$(arg arm_id_2)_link6" reason="Never"/>
-        <disable_collisions link1="$(arg arm_id_2)_leftfinger" link2="$(arg arm_id_2)_link7" reason="Never"/>
         <disable_collisions link1="$(arg arm_id_2)_leftfinger" link2="$(arg arm_id_2)_rightfinger" reason="Default"/>
-        <disable_collisions link1="$(arg arm_id_2)_link3" link2="$(arg arm_id_2)_rightfinger" reason="Never"/>
-        <disable_collisions link1="$(arg arm_id_2)_link4" link2="$(arg arm_id_2)_rightfinger" reason="Never"/>
-        <disable_collisions link1="$(arg arm_id_2)_link6" link2="$(arg arm_id_2)_rightfinger" reason="Never"/>
-        <disable_collisions link1="$(arg arm_id_2)_link7" link2="$(arg arm_id_2)_rightfinger" reason="Never"/>
-        <disable_collisions link1="$(arg arm_id_2)_hand" link2="$(arg arm_id_2)_link3" reason="Never"/>
-        <disable_collisions link1="$(arg arm_id_2)_hand" link2="$(arg arm_id_2)_link4" reason="Never"/>
-        <disable_collisions link1="$(arg arm_id_2)_hand" link2="$(arg arm_id_2)_link6" reason="Never"/>
-        <disable_collisions link1="$(arg arm_id_2)_hand" link2="$(arg arm_id_2)_link7" reason="Adjacent"/>
     </xacro:if>
     <xacro:if value="${hand_2 == 'gamma'}">
-        <disable_collisions link1="$(arg arm_id_2)_ft" link2="$(arg arm_id_2)_link7" reason="Adjacent"/>
         <disable_collisions link1="$(arg arm_id_2)_ft" link2="$(arg arm_id_2)_link7_sc" reason="Adjacent"/>
     </xacro:if>
     <xacro:if value="${hand_2 == 'sponge_eef'}">
-        <disable_collisions link1="$(arg arm_id_2)_ft" link2="$(arg arm_id_2)_link7" reason="Adjacent"/>
         <disable_collisions link1="$(arg arm_id_2)_ft" link2="$(arg arm_id_2)_link7_sc" reason="Adjacent"/>
         <disable_collisions link1="$(arg arm_id_2)_ft" link2="$(arg arm_id_2)_mount" reason="Adjacent"/>
     </xacro:if>
     <xacro:if value="${hand_2 == 'sponge_eef_extend'}">
-        <disable_collisions link1="$(arg arm_id_2)_ft" link2="$(arg arm_id_2)_link7" reason="Adjacent"/>
         <disable_collisions link1="$(arg arm_id_2)_ft" link2="$(arg arm_id_2)_link7_sc" reason="Adjacent"/>
         <disable_collisions link1="$(arg arm_id_2)_ft" link2="$(arg arm_id_2)_mount_extend" reason="Adjacent"/>
         <disable_collisions link1="$(arg arm_id_2)_mount_extend" link2="$(arg arm_id_2)_mount" reason="Adjacent"/>
     </xacro:if>
-    <disable_collisions link1="base" link2="panda_1_link0" reason="Adjacent"/>
-    <disable_collisions link1="base" link2="panda_1_link0_sc" reason="Default"/>
-    <disable_collisions link1="base" link2="panda_1_link1" reason="Never"/>
-    <disable_collisions link1="base" link2="panda_1_link1_sc" reason="Default"/>
-    <disable_collisions link1="base" link2="panda_1_link2" reason="Never"/>
-    <disable_collisions link1="base" link2="panda_1_link2_sc" reason="Never"/>
-    <disable_collisions link1="base" link2="panda_1_link3" reason="Never"/>
-    <disable_collisions link1="base" link2="panda_1_link3_sc" reason="Never"/>
-    <disable_collisions link1="base" link2="panda_1_link4_sc" reason="Never"/>
-    <disable_collisions link1="base" link2="panda_2_link0" reason="Adjacent"/>
-    <disable_collisions link1="base" link2="panda_2_link0_sc" reason="Default"/>
-    <disable_collisions link1="base" link2="panda_2_link1" reason="Never"/>
-    <disable_collisions link1="base" link2="panda_2_link1_sc" reason="Default"/>
-    <disable_collisions link1="base" link2="panda_2_link2" reason="Never"/>
-    <disable_collisions link1="base" link2="panda_2_link2_sc" reason="Never"/>
-    <disable_collisions link1="base" link2="panda_2_link3" reason="Never"/>
-    <disable_collisions link1="base" link2="panda_2_link3_sc" reason="Never"/>
-    <disable_collisions link1="base" link2="panda_2_link4" reason="Never"/>
-    <disable_collisions link1="base" link2="panda_2_link4_sc" reason="Never"/>
-    <disable_collisions link1="panda_1_link0" link2="panda_1_link0_sc" reason="Adjacent"/>
-    <disable_collisions link1="panda_1_link0" link2="panda_1_link1" reason="Adjacent"/>
-    <disable_collisions link1="panda_1_link0" link2="panda_1_link1_sc" reason="Default"/>
-    <disable_collisions link1="panda_1_link0" link2="panda_1_link2" reason="Never"/>
-    <disable_collisions link1="panda_1_link0" link2="panda_1_link2_sc" reason="Never"/>
-    <disable_collisions link1="panda_1_link0" link2="panda_1_link3" reason="Never"/>
-    <disable_collisions link1="panda_1_link0" link2="panda_1_link3_sc" reason="Never"/>
-    <disable_collisions link1="panda_1_link0" link2="panda_1_link4" reason="Never"/>
-    <disable_collisions link1="panda_1_link0" link2="panda_1_link4_sc" reason="Never"/>
-    <disable_collisions link1="panda_1_link0" link2="panda_2_link0" reason="Never"/>
-    <disable_collisions link1="panda_1_link0" link2="panda_2_link0_sc" reason="Never"/>
-    <disable_collisions link1="panda_1_link0" link2="panda_2_link1" reason="Never"/>
-    <disable_collisions link1="panda_1_link0" link2="panda_2_link1_sc" reason="Never"/>
-    <disable_collisions link1="panda_1_link0" link2="panda_2_link2" reason="Never"/>
-    <disable_collisions link1="panda_1_link0" link2="panda_2_link2_sc" reason="Never"/>
-    <disable_collisions link1="panda_1_link0" link2="panda_2_link3" reason="Never"/>
-    <disable_collisions link1="panda_1_link0" link2="panda_2_link3_sc" reason="Never"/>
-    <disable_collisions link1="panda_1_link0" link2="panda_2_link4" reason="Never"/>
-    <disable_collisions link1="panda_1_link0" link2="panda_2_link4_sc" reason="Never"/>
-    <disable_collisions link1="panda_1_link0_sc" link2="panda_1_link1" reason="Never"/>
-    <disable_collisions link1="panda_1_link0_sc" link2="panda_1_link1_sc" reason="Default"/>
-    <disable_collisions link1="panda_1_link0_sc" link2="panda_1_link2" reason="Never"/>
-    <disable_collisions link1="panda_1_link0_sc" link2="panda_1_link2_sc" reason="Never"/>
-    <disable_collisions link1="panda_1_link0_sc" link2="panda_1_link3" reason="Never"/>
-    <disable_collisions link1="panda_1_link0_sc" link2="panda_1_link3_sc" reason="Never"/>
-    <disable_collisions link1="panda_1_link0_sc" link2="panda_1_link4" reason="Never"/>
-    <disable_collisions link1="panda_1_link0_sc" link2="panda_1_link4_sc" reason="Never"/>
-    <disable_collisions link1="panda_1_link0_sc" link2="panda_2_link0" reason="Never"/>
-    <disable_collisions link1="panda_1_link0_sc" link2="panda_2_link0_sc" reason="Never"/>
-    <disable_collisions link1="panda_1_link0_sc" link2="panda_2_link1" reason="Never"/>
-    <disable_collisions link1="panda_1_link0_sc" link2="panda_2_link1_sc" reason="Never"/>
-    <disable_collisions link1="panda_1_link0_sc" link2="panda_2_link2" reason="Never"/>
-    <disable_collisions link1="panda_1_link0_sc" link2="panda_2_link2_sc" reason="Never"/>
-    <disable_collisions link1="panda_1_link0_sc" link2="panda_2_link3" reason="Never"/>
-    <disable_collisions link1="panda_1_link0_sc" link2="panda_2_link3_sc" reason="Never"/>
-    <disable_collisions link1="panda_1_link0_sc" link2="panda_2_link4" reason="Never"/>
-    <disable_collisions link1="panda_1_link0_sc" link2="panda_2_link4_sc" reason="Never"/>
-    <disable_collisions link1="panda_1_link1" link2="panda_1_link1_sc" reason="Adjacent"/>
-    <disable_collisions link1="panda_1_link1" link2="panda_1_link2" reason="Adjacent"/>
-    <disable_collisions link1="panda_1_link1" link2="panda_1_link2_sc" reason="Default"/>
-    <disable_collisions link1="panda_1_link1" link2="panda_1_link3" reason="Never"/>
-    <disable_collisions link1="panda_1_link1" link2="panda_1_link3_sc" reason="Default"/>
-    <disable_collisions link1="panda_1_link1" link2="panda_1_link4" reason="Never"/>
-    <disable_collisions link1="panda_1_link1" link2="panda_1_link4_sc" reason="Never"/>
-    <disable_collisions link1="panda_1_link1" link2="panda_2_link0" reason="Never"/>
-    <disable_collisions link1="panda_1_link1" link2="panda_2_link0_sc" reason="Never"/>
-    <disable_collisions link1="panda_1_link1" link2="panda_2_link1" reason="Never"/>
-    <disable_collisions link1="panda_1_link1" link2="panda_2_link1_sc" reason="Never"/>
-    <disable_collisions link1="panda_1_link1" link2="panda_2_link2" reason="Never"/>
-    <disable_collisions link1="panda_1_link1" link2="panda_2_link2_sc" reason="Never"/>
-    <disable_collisions link1="panda_1_link1" link2="panda_2_link3" reason="Never"/>
-    <disable_collisions link1="panda_1_link1" link2="panda_2_link3_sc" reason="Never"/>
-    <disable_collisions link1="panda_1_link1" link2="panda_2_link4_sc" reason="Never"/>
-    <disable_collisions link1="panda_1_link1_sc" link2="panda_1_link2" reason="Default"/>
-    <disable_collisions link1="panda_1_link1_sc" link2="panda_1_link2_sc" reason="Default"/>
-    <disable_collisions link1="panda_1_link1_sc" link2="panda_1_link3" reason="Never"/>
-    <disable_collisions link1="panda_1_link1_sc" link2="panda_1_link3_sc" reason="Never"/>
-    <disable_collisions link1="panda_1_link1_sc" link2="panda_1_link4" reason="Never"/>
-    <disable_collisions link1="panda_1_link1_sc" link2="panda_1_link4_sc" reason="Never"/>
-    <disable_collisions link1="panda_1_link1_sc" link2="panda_2_link0" reason="Never"/>
-    <disable_collisions link1="panda_1_link1_sc" link2="panda_2_link0_sc" reason="Never"/>
-    <disable_collisions link1="panda_1_link1_sc" link2="panda_2_link1" reason="Never"/>
-    <disable_collisions link1="panda_1_link1_sc" link2="panda_2_link1_sc" reason="Never"/>
-    <disable_collisions link1="panda_1_link1_sc" link2="panda_2_link2" reason="Never"/>
-    <disable_collisions link1="panda_1_link1_sc" link2="panda_2_link2_sc" reason="Never"/>
-    <disable_collisions link1="panda_1_link1_sc" link2="panda_2_link3" reason="Never"/>
-    <disable_collisions link1="panda_1_link1_sc" link2="panda_2_link3_sc" reason="Never"/>
-    <disable_collisions link1="panda_1_link1_sc" link2="panda_2_link4_sc" reason="Never"/>
-    <disable_collisions link1="panda_1_link2" link2="panda_1_link2_sc" reason="Adjacent"/>
-    <disable_collisions link1="panda_1_link2" link2="panda_1_link3" reason="Adjacent"/>
-    <disable_collisions link1="panda_1_link2" link2="panda_1_link3_sc" reason="Default"/>
-    <disable_collisions link1="panda_1_link2" link2="panda_1_link4" reason="Never"/>
-    <disable_collisions link1="panda_1_link2" link2="panda_1_link4_sc" reason="Never"/>
-    <disable_collisions link1="panda_1_link2" link2="panda_2_link0" reason="Never"/>
-    <disable_collisions link1="panda_1_link2" link2="panda_2_link0_sc" reason="Never"/>
-    <disable_collisions link1="panda_1_link2" link2="panda_2_link1" reason="Never"/>
-    <disable_collisions link1="panda_1_link2" link2="panda_2_link1_sc" reason="Never"/>
-    <disable_collisions link1="panda_1_link2" link2="panda_2_link2" reason="Never"/>
-    <disable_collisions link1="panda_1_link2" link2="panda_2_link2_sc" reason="Never"/>
-    <disable_collisions link1="panda_1_link2" link2="panda_2_link3_sc" reason="Never"/>
-    <disable_collisions link1="panda_1_link2_sc" link2="panda_1_link3" reason="Never"/>
-    <disable_collisions link1="panda_1_link2_sc" link2="panda_1_link3_sc" reason="Default"/>
-    <disable_collisions link1="panda_1_link2_sc" link2="panda_1_link4" reason="Never"/>
-    <disable_collisions link1="panda_1_link2_sc" link2="panda_1_link4_sc" reason="Never"/>
-    <disable_collisions link1="panda_1_link2_sc" link2="panda_2_link0" reason="Never"/>
-    <disable_collisions link1="panda_1_link2_sc" link2="panda_2_link0_sc" reason="Never"/>
-    <disable_collisions link1="panda_1_link2_sc" link2="panda_2_link1" reason="Never"/>
-    <disable_collisions link1="panda_1_link2_sc" link2="panda_2_link1_sc" reason="Never"/>
-    <disable_collisions link1="panda_1_link2_sc" link2="panda_2_link2" reason="Never"/>
-    <disable_collisions link1="panda_1_link2_sc" link2="panda_2_link2_sc" reason="Never"/>
-    <disable_collisions link1="panda_1_link2_sc" link2="panda_2_link3" reason="Never"/>
-    <disable_collisions link1="panda_1_link2_sc" link2="panda_2_link3_sc" reason="Never"/>
-    <disable_collisions link1="panda_1_link2_sc" link2="panda_2_link4_sc" reason="Never"/>
-    <disable_collisions link1="panda_1_link3" link2="panda_1_link3_sc" reason="Adjacent"/>
-    <disable_collisions link1="panda_1_link3" link2="panda_1_link4" reason="Adjacent"/>
-    <disable_collisions link1="panda_1_link3" link2="panda_1_link4_sc" reason="Always"/>
-    <disable_collisions link1="panda_1_link3" link2="panda_1_link5" reason="Never"/>
-    <disable_collisions link1="panda_1_link3" link2="panda_1_link5_sc" reason="Always"/>
-    <disable_collisions link1="panda_1_link3" link2="panda_1_link6" reason="Never"/>
-    <disable_collisions link1="panda_1_link3" link2="panda_1_link6_sc" reason="Never"/>
-    <disable_collisions link1="panda_1_link3" link2="panda_1_link7" reason="Never"/>
-    <disable_collisions link1="panda_1_link3" link2="panda_1_link7_sc" reason="Never"/>
-    <disable_collisions link1="panda_1_link3" link2="panda_2_link0" reason="Never"/>
-    <disable_collisions link1="panda_1_link3" link2="panda_2_link0_sc" reason="Never"/>
-    <disable_collisions link1="panda_1_link3" link2="panda_2_link1" reason="Never"/>
-    <disable_collisions link1="panda_1_link3" link2="panda_2_link1_sc" reason="Never"/>
-    <disable_collisions link1="panda_1_link3" link2="panda_2_link2_sc" reason="Never"/>
-    <disable_collisions link1="panda_1_link3_sc" link2="panda_1_link4" reason="Always"/>
-    <disable_collisions link1="panda_1_link3_sc" link2="panda_1_link4_sc" reason="Always"/>
-    <disable_collisions link1="panda_1_link3_sc" link2="panda_1_link5" reason="Never"/>
-    <disable_collisions link1="panda_1_link3_sc" link2="panda_1_link5_sc" reason="Never"/>
-    <disable_collisions link1="panda_1_link3_sc" link2="panda_1_link6" reason="Never"/>
-    <disable_collisions link1="panda_1_link3_sc" link2="panda_1_link6_sc" reason="Never"/>
-    <disable_collisions link1="panda_1_link3_sc" link2="panda_1_link7" reason="Never"/>
-    <disable_collisions link1="panda_1_link3_sc" link2="panda_1_link7_sc" reason="Never"/>
-    <disable_collisions link1="panda_1_link3_sc" link2="panda_2_link0" reason="Never"/>
-    <disable_collisions link1="panda_1_link3_sc" link2="panda_2_link0_sc" reason="Never"/>
-    <disable_collisions link1="panda_1_link3_sc" link2="panda_2_link1" reason="Never"/>
-    <disable_collisions link1="panda_1_link3_sc" link2="panda_2_link1_sc" reason="Never"/>
-    <disable_collisions link1="panda_1_link3_sc" link2="panda_2_link2" reason="Never"/>
-    <disable_collisions link1="panda_1_link3_sc" link2="panda_2_link2_sc" reason="Never"/>
-    <disable_collisions link1="panda_1_link4" link2="panda_1_link4_sc" reason="Adjacent"/>
-    <disable_collisions link1="panda_1_link4" link2="panda_1_link5" reason="Adjacent"/>
-    <disable_collisions link1="panda_1_link4" link2="panda_1_link5_sc" reason="Always"/>
-    <disable_collisions link1="panda_1_link4" link2="panda_1_link6" reason="Never"/>
-    <disable_collisions link1="panda_1_link4" link2="panda_1_link6_sc" reason="Never"/>
-    <disable_collisions link1="panda_1_link4" link2="panda_1_link7" reason="Never"/>
-    <disable_collisions link1="panda_1_link4" link2="panda_1_link7_sc" reason="Never"/>
-    <disable_collisions link1="panda_1_link4" link2="panda_2_link0" reason="Never"/>
-    <disable_collisions link1="panda_1_link4" link2="panda_2_link0_sc" reason="Never"/>
-    <disable_collisions link1="panda_1_link4_sc" link2="panda_1_link5" reason="Never"/>
-    <disable_collisions link1="panda_1_link4_sc" link2="panda_1_link5_sc" reason="Always"/>
-    <disable_collisions link1="panda_1_link4_sc" link2="panda_1_link6" reason="Never"/>
-    <disable_collisions link1="panda_1_link4_sc" link2="panda_1_link6_sc" reason="Never"/>
-    <disable_collisions link1="panda_1_link4_sc" link2="panda_1_link7" reason="Never"/>
-    <disable_collisions link1="panda_1_link4_sc" link2="panda_1_link7_sc" reason="Never"/>
-    <disable_collisions link1="panda_1_link4_sc" link2="panda_2_link0" reason="Never"/>
-    <disable_collisions link1="panda_1_link4_sc" link2="panda_2_link0_sc" reason="Never"/>
-    <disable_collisions link1="panda_1_link4_sc" link2="panda_2_link1" reason="Never"/>
-    <disable_collisions link1="panda_1_link4_sc" link2="panda_2_link1_sc" reason="Never"/>
-    <disable_collisions link1="panda_1_link4_sc" link2="panda_2_link2_sc" reason="Never"/>
-    <disable_collisions link1="panda_1_link5" link2="panda_1_link5_sc" reason="Adjacent"/>
-    <disable_collisions link1="panda_1_link5" link2="panda_1_link6" reason="Adjacent"/>
-    <disable_collisions link1="panda_1_link5" link2="panda_1_link6_sc" reason="Always"/>
-    <disable_collisions link1="panda_1_link5" link2="panda_2_link5" reason="Default"/>
-    <disable_collisions link1="panda_1_link5" link2="panda_2_link5_sc" reason="Default"/>
-    <disable_collisions link1="panda_1_link5" link2="panda_2_link6_sc" reason="Default"/>
-    <disable_collisions link1="panda_1_link5_sc" link2="panda_1_link6" reason="Never"/>
-    <disable_collisions link1="panda_1_link5_sc" link2="panda_1_link6_sc" reason="Always"/>
-    <disable_collisions link1="panda_1_link5_sc" link2="panda_1_link7" reason="Never"/>
-    <disable_collisions link1="panda_1_link5_sc" link2="panda_1_link7_sc" reason="Never"/>
-    <disable_collisions link1="panda_1_link5_sc" link2="panda_2_link5_sc" reason="Default"/>
-    <disable_collisions link1="panda_1_link6" link2="panda_1_link6_sc" reason="Adjacent"/>
-    <disable_collisions link1="panda_1_link6" link2="panda_1_link7" reason="Adjacent"/>
-    <disable_collisions link1="panda_1_link6" link2="panda_1_link7_sc" reason="Default"/>
-    <disable_collisions link1="panda_1_link6" link2="panda_2_link5_sc" reason="Default"/>
-    <disable_collisions link1="panda_1_link6" link2="panda_2_link7_sc" reason="Default"/>
-    <disable_collisions link1="panda_1_link6_sc" link2="panda_1_link7" reason="Never"/>
-    <disable_collisions link1="panda_1_link6_sc" link2="panda_1_link7_sc" reason="Default"/>
-    <disable_collisions link1="panda_1_link6_sc" link2="panda_2_link5_sc" reason="Default"/>
-    <disable_collisions link1="panda_1_link6_sc" link2="panda_2_link6" reason="Default"/>
-    <disable_collisions link1="panda_1_link6_sc" link2="panda_2_link6_sc" reason="Default"/>
-    <disable_collisions link1="panda_1_link7" link2="panda_1_link7_sc" reason="Adjacent"/>
-    <disable_collisions link1="panda_1_link7_sc" link2="panda_2_link5" reason="Default"/>
-    <disable_collisions link1="panda_1_link7_sc" link2="panda_2_link5_sc" reason="Default"/>
-    <disable_collisions link1="panda_1_link7_sc" link2="panda_2_link7_sc" reason="Default"/>
-    <disable_collisions link1="panda_2_link0" link2="panda_2_link0_sc" reason="Adjacent"/>
-    <disable_collisions link1="panda_2_link0" link2="panda_2_link1" reason="Adjacent"/>
-    <disable_collisions link1="panda_2_link0" link2="panda_2_link1_sc" reason="Default"/>
-    <disable_collisions link1="panda_2_link0" link2="panda_2_link2" reason="Never"/>
-    <disable_collisions link1="panda_2_link0" link2="panda_2_link2_sc" reason="Never"/>
-    <disable_collisions link1="panda_2_link0" link2="panda_2_link3" reason="Never"/>
-    <disable_collisions link1="panda_2_link0" link2="panda_2_link3_sc" reason="Never"/>
-    <disable_collisions link1="panda_2_link0" link2="panda_2_link4" reason="Never"/>
-    <disable_collisions link1="panda_2_link0" link2="panda_2_link4_sc" reason="Never"/>
-    <disable_collisions link1="panda_2_link0_sc" link2="panda_2_link1" reason="Never"/>
-    <disable_collisions link1="panda_2_link0_sc" link2="panda_2_link1_sc" reason="Default"/>
-    <disable_collisions link1="panda_2_link0_sc" link2="panda_2_link2" reason="Never"/>
-    <disable_collisions link1="panda_2_link0_sc" link2="panda_2_link2_sc" reason="Never"/>
-    <disable_collisions link1="panda_2_link0_sc" link2="panda_2_link3" reason="Never"/>
-    <disable_collisions link1="panda_2_link0_sc" link2="panda_2_link3_sc" reason="Never"/>
-    <disable_collisions link1="panda_2_link0_sc" link2="panda_2_link4" reason="Never"/>
-    <disable_collisions link1="panda_2_link0_sc" link2="panda_2_link4_sc" reason="Never"/>
-    <disable_collisions link1="panda_2_link1" link2="panda_2_link1_sc" reason="Adjacent"/>
-    <disable_collisions link1="panda_2_link1" link2="panda_2_link2" reason="Adjacent"/>
-    <disable_collisions link1="panda_2_link1" link2="panda_2_link2_sc" reason="Default"/>
-    <disable_collisions link1="panda_2_link1" link2="panda_2_link3" reason="Never"/>
-    <disable_collisions link1="panda_2_link1" link2="panda_2_link3_sc" reason="Default"/>
-    <disable_collisions link1="panda_2_link1" link2="panda_2_link4" reason="Never"/>
-    <disable_collisions link1="panda_2_link1" link2="panda_2_link4_sc" reason="Never"/>
-    <disable_collisions link1="panda_2_link1_sc" link2="panda_2_link2" reason="Default"/>
-    <disable_collisions link1="panda_2_link1_sc" link2="panda_2_link2_sc" reason="Default"/>
-    <disable_collisions link1="panda_2_link1_sc" link2="panda_2_link3" reason="Never"/>
-    <disable_collisions link1="panda_2_link1_sc" link2="panda_2_link4" reason="Never"/>
-    <disable_collisions link1="panda_2_link1_sc" link2="panda_2_link4_sc" reason="Never"/>
-    <disable_collisions link1="panda_2_link2" link2="panda_2_link2_sc" reason="Adjacent"/>
-    <disable_collisions link1="panda_2_link2" link2="panda_2_link3" reason="Adjacent"/>
-    <disable_collisions link1="panda_2_link2" link2="panda_2_link3_sc" reason="Default"/>
-    <disable_collisions link1="panda_2_link2" link2="panda_2_link4" reason="Never"/>
-    <disable_collisions link1="panda_2_link2" link2="panda_2_link4_sc" reason="Never"/>
-    <disable_collisions link1="panda_2_link2_sc" link2="panda_2_link3" reason="Never"/>
-    <disable_collisions link1="panda_2_link2_sc" link2="panda_2_link3_sc" reason="Default"/>
-    <disable_collisions link1="panda_2_link2_sc" link2="panda_2_link4" reason="Never"/>
-    <disable_collisions link1="panda_2_link2_sc" link2="panda_2_link4_sc" reason="Never"/>
-    <disable_collisions link1="panda_2_link3" link2="panda_2_link3_sc" reason="Adjacent"/>
-    <disable_collisions link1="panda_2_link3" link2="panda_2_link4" reason="Adjacent"/>
-    <disable_collisions link1="panda_2_link3" link2="panda_2_link4_sc" reason="Always"/>
-    <disable_collisions link1="panda_2_link3" link2="panda_2_link5" reason="Never"/>
-    <disable_collisions link1="panda_2_link3" link2="panda_2_link5_sc" reason="Always"/>
-    <disable_collisions link1="panda_2_link3" link2="panda_2_link6" reason="Never"/>
-    <disable_collisions link1="panda_2_link3" link2="panda_2_link6_sc" reason="Never"/>
-    <disable_collisions link1="panda_2_link3" link2="panda_2_link7" reason="Never"/>
-    <disable_collisions link1="panda_2_link3" link2="panda_2_link7_sc" reason="Never"/>
-    <disable_collisions link1="panda_2_link3_sc" link2="panda_2_link4" reason="Always"/>
-    <disable_collisions link1="panda_2_link3_sc" link2="panda_2_link4_sc" reason="Always"/>
-    <disable_collisions link1="panda_2_link3_sc" link2="panda_2_link5" reason="Never"/>
-    <disable_collisions link1="panda_2_link3_sc" link2="panda_2_link5_sc" reason="Never"/>
-    <disable_collisions link1="panda_2_link3_sc" link2="panda_2_link6" reason="Never"/>
-    <disable_collisions link1="panda_2_link3_sc" link2="panda_2_link6_sc" reason="Never"/>
-    <disable_collisions link1="panda_2_link3_sc" link2="panda_2_link7" reason="Never"/>
-    <disable_collisions link1="panda_2_link3_sc" link2="panda_2_link7_sc" reason="Never"/>
-    <disable_collisions link1="panda_2_link4" link2="panda_2_link4_sc" reason="Adjacent"/>
-    <disable_collisions link1="panda_2_link4" link2="panda_2_link5" reason="Adjacent"/>
-    <disable_collisions link1="panda_2_link4" link2="panda_2_link5_sc" reason="Default"/>
-    <disable_collisions link1="panda_2_link4" link2="panda_2_link6" reason="Never"/>
-    <disable_collisions link1="panda_2_link4" link2="panda_2_link6_sc" reason="Never"/>
-    <disable_collisions link1="panda_2_link4" link2="panda_2_link7" reason="Never"/>
-    <disable_collisions link1="panda_2_link4" link2="panda_2_link7_sc" reason="Never"/>
-    <disable_collisions link1="panda_2_link4_sc" link2="panda_2_link5" reason="Never"/>
-    <disable_collisions link1="panda_2_link4_sc" link2="panda_2_link5_sc" reason="Default"/>
-    <disable_collisions link1="panda_2_link4_sc" link2="panda_2_link6" reason="Never"/>
-    <disable_collisions link1="panda_2_link4_sc" link2="panda_2_link6_sc" reason="Never"/>
-    <disable_collisions link1="panda_2_link4_sc" link2="panda_2_link7" reason="Never"/>
-    <disable_collisions link1="panda_2_link4_sc" link2="panda_2_link7_sc" reason="Never"/>
-    <disable_collisions link1="panda_2_link5" link2="panda_2_link5_sc" reason="Adjacent"/>
-    <disable_collisions link1="panda_2_link5" link2="panda_2_link6" reason="Adjacent"/>
-    <disable_collisions link1="panda_2_link5" link2="panda_2_link6_sc" reason="Default"/>
-    <disable_collisions link1="panda_2_link5_sc" link2="panda_2_link6" reason="Never"/>
-    <disable_collisions link1="panda_2_link5_sc" link2="panda_2_link6_sc" reason="Default"/>
-    <disable_collisions link1="panda_2_link5_sc" link2="panda_2_link7" reason="Never"/>
-    <disable_collisions link1="panda_2_link5_sc" link2="panda_2_link7_sc" reason="Never"/>
-    <disable_collisions link1="panda_2_link6" link2="panda_2_link6_sc" reason="Adjacent"/>
-    <disable_collisions link1="panda_2_link6" link2="panda_2_link7" reason="Adjacent"/>
-    <disable_collisions link1="panda_2_link6" link2="panda_2_link7_sc" reason="Default"/>
-    <disable_collisions link1="panda_2_link6_sc" link2="panda_2_link7" reason="Never"/>
-    <disable_collisions link1="panda_2_link6_sc" link2="panda_2_link7_sc" reason="Default"/>
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