Commit message: Setup single arm control + planning.

File: mmint_franka_description/robots/panda.urdf (robot description, URDF)
Before this commit: robot panda, 41 links, 40 joints
Links:
- removed link panda_2_link0
- removed link panda_2_link0_sc
- removed link panda_2_link1
- removed link panda_2_link1_sc
- removed link panda_2_link2
- removed link panda_2_link2_sc
- removed link panda_2_link3
- removed link panda_2_link3_sc
- removed link panda_2_link4
- removed link panda_2_link4_sc
- removed link panda_2_link5
- removed link panda_2_link5_sc
- removed link panda_2_link6
- removed link panda_2_link6_sc
- removed link panda_2_link7
- removed link panda_2_link7_sc
- removed link panda_2_link8
Joints:
- removed joint panda_2_joint1
- removed joint panda_2_joint2
- removed joint panda_2_joint3
- removed joint panda_2_joint4
- removed joint panda_2_joint5
- removed joint panda_2_joint6
- removed joint panda_2_joint7
- removed joint panda_2_joint8
- removed joint panda_2_joint_base
- removed joint panda_2_link0_sc_joint
- removed joint panda_2_link1_sc_joint
- removed joint panda_2_link2_sc_joint
- removed joint panda_2_link3_sc_joint
- removed joint panda_2_link4_sc_joint
- removed joint panda_2_link5_sc_joint
- removed joint panda_2_link6_sc_joint
- removed joint panda_2_link7_sc_joint
- joint panda_1_joint_base: origin xyz=0.0 0.4425 0.6 rpy=0.0 0.0 -1.57079633 -> xyz=0 0.4425 0.6 rpy=0.0 0.0 -1.57079633
