Commit message: Fix bug that applied offset to wrist camera connection in the wrong case

File: mmint_franka_description/robots/mmint_panda.urdf.xacro (robot description, xacro)
@@ -59,8 +59,8 @@
     <xacro:if value="${include_wrist_camera}">
         <xacro:if value="${include_gamma}">
-            <xacro:wrist_camera ns="$(arg arm_id)" connected_to="$(arg arm_id)_ft_origin"/>
+            <xacro:wrist_camera ns="$(arg arm_id)" xyz="0 0 0.0079" connected_to="$(arg arm_id)_ft_origin"/>
         </xacro:if>
         <xacro:unless value="${include_gamma}">
-            <xacro:wrist_camera ns="$(arg arm_id)" xyz="0 0 0.0079" connected_to="$(arg arm_id)_flange"/>
+            <xacro:wrist_camera ns="$(arg arm_id)" connected_to="$(arg arm_id)_flange"/>
         </xacro:unless>
         <xacro:property name="connecting_link" value="$(arg arm_id)_wrist_camera_flange"/>

File: mmint_franka_description/robots/panda_gelsight.urdf (robot description, URDF)
Before this commit: robot panda, 35 links, 34 joints
Links:
- added link panda_1_flange
- added link panda_1_wrist_camera_flange
- added link panda_1_wrist_camera_frame
- added link panda_1_wrist_camera_mount
Joints:
- added joint panda_1_flange_joint: type fixed, parent panda_1_link8, child panda_1_flange, origin rpy=0 0 -0.7853981633974483
- added joint panda_1_wrist_camera_flange_joint: type fixed, parent panda_1_wrist_camera_mount, child panda_1_wrist_camera_flange, origin xyz=0 0 0.0018 rpy=0 0 0
- added joint panda_1_wrist_camera_frame_joint: type fixed, parent panda_1_wrist_camera_mount, child panda_1_wrist_camera_frame, origin xyz=0.1 0.01 0.025 rpy=0.6283185305473132 0 -1.5707963267948968
- added joint panda_1_wrist_camera_joint: type fixed, parent panda_1_ft_origin, child panda_1_wrist_camera_mount, origin xyz=0 0 0 rpy=0 0 0
- joint elastomer_joint_left: origin xyz=0.0 0.0 0.0 rpy=0 0 0 -> xyz=0.0 0.0 -0.0054 rpy=0 0 0; parent panda_1_fingerbox_left -> panda_1_leftfinger
- joint elastomer_joint_right: origin xyz=0.0 0.0 0.0 rpy=0 0 0 -> xyz=0.0 0.0 -0.0054 rpy=0 0 0
- joint panda_1_fingerbox_left_joint: origin xyz=0.0 0.0 0.0 rpy=0 0 0 -> xyz=0.0 0.0 -0.0054 rpy=0 0 0
- joint panda_1_fingerbox_right_joint: origin xyz=0.0 0.0 0.0 rpy=0 0 0 -> xyz=0.0 0.0 -0.0054 rpy=0 0 0
- joint panda_1_ft_joint: origin xyz=0 0 0 rpy=0 0 -0.7853981633974483 -> xyz=0 0 0 rpy=0 0 0; parent panda_1_link8 -> panda_1_flange
- joint panda_1_hand_joint: origin xyz=0 0 0.0079 rpy=0 0 0 -> xyz=0 0 0 rpy=0 0 0; parent panda_1_ft_origin -> panda_1_wrist_camera_flange
