Commit message: Setup switch joint position

File: mmint_franka_single_moveit_config/config/panda.srdf.xacro (robot description, xacro)
@@ -25,4 +25,13 @@
         <joint name="$(arg arm_id)_joint6" value="${pi/2}"/>
         <joint name="$(arg arm_id)_joint7" value="${pi/4}"/>
+    </group_state>
+    <group_state name="switch_eef" group="$(arg arm_id)">
+        <joint name="$(arg arm_id)_joint1" value="1.885"/>
+        <joint name="$(arg arm_id)_joint2" value="0"/>
+        <joint name="$(arg arm_id)_joint3" value="0"/>
+        <joint name="$(arg arm_id)_joint4" value="-2.269"/>
+        <joint name="$(arg arm_id)_joint5" value="0"/>
+        <joint name="$(arg arm_id)_joint6" value="2.95"/>
+        <joint name="$(arg arm_id)_joint7" value="0.768"/>
     </group_state>
     <!--DISABLE COLLISIONS: By default it is assumed that any link of the robot could potentially come into collision with any other link in the robot. This tag disables collision checking between a specified pair of links. -->

Commit message: Update the srdf for new urdf parameterization

File: mmint_franka_single_moveit_config/config/panda.srdf.xacro (robot description, xacro)
@@ -7,5 +7,9 @@
     <xacro:arg name="arm_id" default="panda_1"/>
     <xacro:arg name="hand" default="panda_hand"/>
+    <xacro:arg name="include_gamma" default="false"/>
+    <xacro:arg name="include_wrist_camera" default="false"/>
     <xacro:property name="hand" value="$(arg hand)"/>
+    <xacro:property name="include_gamma" value="$(arg include_gamma)"/>
+    <xacro:property name="include_wrist_camera" value="$(arg include_wrist_camera)"/>
     <!--GROUPS: Representation of a set of joints and links. This can be useful for specifying DOF to plan for, defining arms, end effectors, etc-->
     <!--LINKS: When a link is specified, the parent joint of that link (if it exists) is automatically included-->
@@ -74,6 +78,11 @@
     <xacro:configure_collisions arm_id="$(arg arm_id)" link="7"/>
     <xacro:if value="${hand == 'panda_gelsight'}">
-        <xacro:disable_collisions_for link="$(arg arm_id)_ft"
-                                      others="${['$(arg arm_id)_link8', '$(arg arm_id)_hand', '$(arg arm_id)_link7', '$(arg arm_id)_link7_sc']}"/>
+        <xacro:if value="${include_gamma}">
+            <xacro:disable_collisions_for link="$(arg arm_id)_hand" others="${['$(arg arm_id)_ft']}"/>
+        </xacro:if>
+        <xacro:unless value="${include_gamma}">
+            <xacro:disable_collisions_for link="$(arg arm_id)_hand"
+                                          others="${['$(arg arm_id)_link7', '$(arg arm_id)_link7_sc', '$(arg arm_id)_link8']}"/>
+        </xacro:unless>
         <xacro:disable_collisions_for link="$(arg arm_id)_hand"
                                       others="${['mount_left', '$(arg arm_id)_leftfinger', 'mount_right', '$(arg arm_id)_rightfinger']}"/>
@@ -83,20 +92,3 @@
         <xacro:disable_collisions_for link="$(arg arm_id)_rightfinger" others="${['$(arg arm_id)_fingerbox_right']}"/>
     </xacro:if>
-    <xacro:if value="${hand == 'panda_gelsight_no_gamma'}">
-        <xacro:disable_collisions_for link="$(arg arm_id)_hand"
-                                      others="${['$(arg arm_id)_link7', '$(arg arm_id)_link7_sc', '$(arg arm_id)_link8', 'mount_left', '$(arg arm_id)_leftfinger', 'mount_right', '$(arg arm_id)_rightfinger']}"/>
-        <xacro:disable_collisions_for link="mount_left" others="${['$(arg arm_id)_leftfinger']}"/>
-        <xacro:disable_collisions_for link="mount_right" others="${['$(arg arm_id)_rightfinger']}"/>
-        <xacro:disable_collisions_for link="$(arg arm_id)_leftfinger" others="${['$(arg arm_id)_fingerbox_left']}"/>
-        <xacro:disable_collisions_for link="$(arg arm_id)_rightfinger" others="${['$(arg arm_id)_fingerbox_right']}"/>
-    </xacro:if>
-    <xacro:if value="${hand == 'sponge_eef_extend_no_gamma'}">
-        <disable_collisions link1="$(arg arm_id)_ft" link2="$(arg arm_id)_link7_sc" reason="Adjacent"/>
-        <disable_collisions link1="$(arg arm_id)_ft" link2="$(arg arm_id)_mount_extend" reason="Adjacent"/>
-        <disable_collisions link1="$(arg arm_id)_mount_extend" link2="$(arg arm_id)_mount" reason="Adjacent"/>
-    </xacro:if>
-    <xacro:if value="${hand == 'sponge_eef_no_gamma'}">
-        <disable_collisions link1="$(arg arm_id)_ft" link2="$(arg arm_id)_link7_sc" reason="Adjacent"/>
-        <disable_collisions link1="$(arg arm_id)_ft" link2="$(arg arm_id)_mount" reason="Adjacent"/>
-    </xacro:if>
 </robot>
